File: dino_v0_0_1/_autosave-dino_v0_0_1.kicad_sch (KiCad schematic)
At the start: 17 parts, among them SW1 SW_DIP_x07, U1 74LS590, U2 74LS590, U3 NE555P

Commit message: Organizes datasheets and updates schematics
Renames PDF resources into a dedicated 'datasheets' folder
for better organization and clarity. Removes outdated PDFs
to improve project maintainability. Enhances schematic by
adding resistor symbol and adjusting LED positions for
optimized layout. Moves DOCX files to 'docs' directory, keeping
versions clear and manageable.
Parts:
- added R1: R, symbol Device:R
Other:
- moved on the sheet: D1, D2, D3, D4, D5, D6, D7, D8
