File: dino_v0_0_2/data.kicad_sch (KiCad schematic)
At the start: 4 parts

Commit message: DINO Updates
Parts:
- removed Bus-Arbiter1: 74LS645, symbol 74xx:74LS645
- removed HighCounter1, LowCounter1: 74LS590, symbol 74xx:74LS590
- removed MCM60256AP1: SRAM, symbol Memory_RAM:MCM60256AP
Connections:
- no-connect marks 2 -> 0
Other:
- note removed: "Ripple Cascade"
