File: dino_v0_0_2/control_word.kicad_sch (KiCad schematic)
At the start: 4 parts, among them U27 74LS138, U28 74LS138, U29 74LS138, U30 74LS138

Commit message: Schematic Update
Other:
- note added: "[11:9]"
- note added: "[12]"
- note added: "[13]"
- note added: "[14]"
- note added: "[15]"
- note added: "[2:0]"
- note added: "[5:3]"
- note added: "[8:6]"
Changed lines of the file:
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@@
+		)
+	)
+	(text "[15]"
+		(exclude_from_sim no)
+		(at 156.21 133.604 0)
+		(effects
+			(font
+				(size 1.27 1.27)
+			)
 		)
 	)
@@
 		)
 	)
+	(text "[13]"
+		(exclude_from_sim no)
+		(at 157.988 125.984 0)
+		(effects
+			(font
+				(size 1.27 1.27)
+			)
+		)
+	)
 	(text "001"
 		(exclude_from_sim no)
@@
 		)
 	)
+	(text "[14]"
+		(exclude_from_sim no)
+		(at 164.084 129.794 0)
+		(effects
+			(font
+				(size 1.27 1.27)
+			)
+		)
+	)
+	(text "[8:6]"
+		(exclude_from_sim no)
+		(at 163.83 38.354 0)
+		(effects
+			(font
+				(size 1.27 1.27)
+			)
+		)
+	)
 	(text "100"
 		(exclude_from_sim no)
@@
 		)
 	)
+	(text "[2:0]"
+		(exclude_from_sim no)
+		(at 163.83 78.74 0)
+		(effects
+			(font
+				(size 1.27 1.27)
+			)
+		)
+	)
 	(text "001"
 		(exclude_from_sim no)
@@
 		)
 	)
+	(text "[12]"
+		(exclude_from_sim no)
+		(at 163.576 122.174 0)
+		(effects
+			(font
+				(size 1.27 1.27)
+			)
+		)
+	)
 	(text "011"
 		(exclude_from_sim no)
@@
 		)
 	)
+	(text "[11:9]"
+		(exclude_from_sim no)
+		(at 116.586 38.862 0)
+		(effects
+			(font
+				(size 1.27 1.27)
+			)
+		)
+	)
 	(text "010"
 		(exclude_from_sim no)
@@
 		(effects
 			(font
+				(size 1.27 1.27)
+			)
+		)
+	)
+	(text "[5:3]"
+		(exclude_from_sim no)
+		(at 116.84 78.486 0)
+		(effects
+			(font
