File: dino_v0_0_2/control_word.kicad_sch (KiCad schematic)
At the start: 4 parts, among them U27 74LS138, U28 74LS138, U29 74LS138, U30 74LS138

Commit message: v0.3.0 - Rev 1.2.0 Update
Parts:
- removed U27: 74LS138, symbol 74xx:74LS138
Connections:
- net MDR_LOAD is gone; now on net NC: U29.7 (O7)
- net OUR_REG_OUT is gone; now on net NC: U28.7 (O7)
- net SYS_CLK_HALT is gone; now on net NC: U29.10 (O5)
- net NC: no longer U29.12 (O3), U30.7 (O7)
- net MAR_HI_LOAD renamed ~{REG_C_OUT}
- net MAR_LOAD renamed ~{ALU_OUT}
- net MAR_LOW_LOAD renamed ~{REG_B_OUT}
- net MDR_OUT renamed ~{MDR_OUT}
- net NOP renamed NONE
- net OUT_REG_LOAD renamed ~{OUT_REG_LOAD}
- net PC_CLEAR renamed ~{PC_CLEAR}
- net PC_PRESET renamed ~{PC_LOAD}
- net RAM_LOAD renamed ~{REG_A_OUT}
- net RAM_OUT renamed ~{RAM_OUT}
- net REG_A_LOAD renamed ~{REG_A_LOAD}
- net REG_A_OUT renamed ~{MAR_LO_LOAD}
- net REG_B_LOAD renamed ~{REG_B_LOAD}
- net REG_B_OUT renamed ~{MAR_HI_LOAD}
- net REG_C_LOAD renamed ~{REG_C_LOAD}
- net REG_C_OUT renamed ~{IR_LOAD}
- net ROM_OUT renamed ~{ROM_OUT}
- new net ~{COND}: U29.12 (O3)
- new net ~{RAM_LOAD}: U30.7 (O7)
Other:
- note added: "ADD"
- note added: "AND"
- note added: "BSUB"
- note added: "CLR"
- note added: "OR"
- note added: "PC=1 MAR=0"
- note added: "SET"
- note added: "SUB"
- note added: "XOR"
- note added: "[11:9] ALU Bus"
- note removed: "[11:9]"
- title: Dino v0.0.2 -> Dino v0.0.3
