File: dino_v0_0_2/control_word.kicad_sch (KiCad schematic)
At the start: 12 parts, among them U28 74LS138, U29 74LS138, U30 74LS138, U62 74LS02, U70 74LS138, U71 74LS138

Commit message: feat: phase E step A -- the 16K I/O window, in schematic
Carves 0x4000-0x7FFF out of ROM space and publishes a bus. The ROM now
answers 0x0000-0x3FFF only; the window decodes to no core chip, so W
reads its park -- 0xFF, which is HALT.

TWO NEW PACKAGES, both on the memory board:

  U74 '00  ~{M14}      = NAND(M14, M14)
           ~{ROM_SEL}  = NAND(~{RAM_EN}, ~{M14})
           ~{RAM_OE_G} = NAND(RAM_OE_ON, M15)
           ~{IO_SEL}   = NAND(~{RAM_EN}, M14)
  U75 '32  ~{IO_RD}    = OR(~{IO_SEL}, READS_IDLE)
           ~{IO_WR}    = OR(~{IO_SEL}, ~{RAM_WRITE_EN})
           RESET_B     = OR(RESET, GND)
           ~{IO_RD_Q}  = OR(~{IO_RD}, CLK)

Eight copper changes: U24.20 and U22.12 to ~{ROM_SEL}, U26.22/U51.9 fed
from U74 g3, U39.10 to ~{IO_RD}, U37.10 and U28.7 unlanded, U37.11 to
GND. Park: R4-R8 + R25-R27, 4.7k on W0-7. CLK crosses through R3, 100R,
source end -- the R2 treatment.

IN RETIRES. ~{SW_OUT} has zero pins project-wide. SWITCH-GATE1's enables
are strapped +5V until card zero drives them from an address decode.

THE ROM_EN ALIAS IS DELETED. Once U24.20 moved, ROM_EN named a net with
no ROM consumer. Deleting it half-way SPLIT the net and alias_splits()
caught it mid-edit -- M15: ['M15', 'M15/ROM_EN'], the exact two-key
failure that once cost this project the ROM chip-enable on every
continuity checklist ever generated.

CLK WAS A FOURTH CROSSING THE SPEC DID NOT CARRY. Census: 15 CLK pins,
none on the memory board; ~{CLK} at U51.4 is the wrong polarity and both
new packages are full. SECTION 1's cost table predated the read-term
split that spent U75 g4, so memory is +4 and MDR is +4 -- the wire margin
is zero. Ruled: stay on memory, the output-load argument still holds.

SWITCH-GATE1/SW1/R17-R24/C48 move to their own input.kicad_sch so the
DIP card is modelled as a card. No renumbering: 168 designators
unchanged, --since reports annotate=0.

TOOLING RECONCILED TO THE DESIGN, not the reverse:
  test_continuity_completeness  M15_PINS U24.20 -> U74.10; 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
Connections:
- net ~{SW_OUT}: no longer names the net of U28.7 (O7)
- no-connect marks 13 -> 14
Changed lines of the file:
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@@
 	)
 	(no_connect
+		(at 93.98 93.98)
+	)
+	(no_connect
 		(at 220.98 83.82)
 	)
@@
 	(wire
 		(pts
-			(xy 90.17 93.98) (xy 93.98 93.98)
-		)
-		(stroke
-			(width 0)
-			(type default)
-		)
-	)
-	(wire
-		(pts
 			(xy 170.18 83.82) (xy 166.37 83.82)
 		)
@@
 		)
 	)
-	(label "~{SW_OUT}"
-		(at 90.17 93.98 180)
-		(effects
-			(font
-				(size 1.27 1.27)
-			)
-			(justify right bottom)
-		)
-	)
 	(label "CW18"
 		(at 132.08 133.35 0)
@@
 		)
 	)
-	(text "MODULE CONTRACT — generated, do not hand-edit (kicad_contracts.py --stamp)\nIN: FLAG_Z <- ALU Module\nIN: CW0-8, CW17=~{SRC_BANK}, CW18=~{DST_BANK} <- Microcode_Decoder\nOUT: ~{ALU_OUT} -> ALU Module, Memory Data Register\nOUT: ~{REG_A_LOAD}, ~{REG_B_LOAD} -> ALU Module, Register Modules\nOUT: ~{MAR_HI_LOAD}, ~{MAR_LO_LOAD} -> Memory Address Regiser\nOUT: SRC_ACTIVE, ~{IR_LOAD}, ~{MDR_OUT}, ~{PC_HI_OUT}, ~{PC_LO_OUT}, ~{RAM_LOAD}, ~{RAM_OUT} -> Memory Data Register\nOUT: ~{SW_OUT} -> Memory Data Register, Output\nOUT: ~{ROM_OUT} -> Memory, Memory Data Register\nOUT: ~{PC_CLEAR}, ~{PC_LOAD} -> Program Counter\nOUT: ~{REG_A_OUT}, ~{REG_B_OUT}, ~{REG_C_LOAD}, ~{REG_C_OUT}, ~{REG_OUT_LOAD} -> Register Modules\nOUT: ~{SP_DOWN}, ~{SP_HI_LOAD}, ~{SP_HI_OUT}, ~{SP_LO_LOAD}, ~{SP_LO_OUT}, ~{SP_UP} -> Stack Pointer"
+	(text "MODULE CONTRACT — generated, do not hand-edit (kicad_contracts.py --stamp)\nIN: FLAG_Z <- ALU Module\nIN: CW0-8, CW17=~{SRC_BANK}, CW18=~{DST_BANK} <- Microcode_Decoder\nOUT: ~{ALU_OUT} -> ALU Module, Memory Data Register\nOUT: ~{REG_A_LOAD}, ~{REG_B_LOAD} -> ALU Module, Register Modules\nOUT: ~{MAR_HI_LOAD}, ~{MAR_LO_LOAD} -> Memory Address Regiser\nOUT: SRC_ACTIVE, ~{IR_LOAD}, ~{MDR_OUT}, ~{PC_HI_OUT}, ~{PC_LO_OUT}, ~{RAM_LOAD}, ~{RAM_OUT} -> Memory Data Register\nOUT: ~{ROM_OUT} -> Memory, Memory Data Register\nOUT: ~{PC_CLEAR}, ~{PC_LOAD} -> Program Counter\nOUT: ~{REG_A_OUT}, ~{REG_B_OUT}, ~{REG_C_LOAD}, ~{REG_C_OUT}, ~{REG_OUT_LOAD} -> Register Modules\nOUT: ~{SP_DOWN}, ~{SP_HI_LOAD}, ~{SP_HI_OUT}, ~{SP_LO_LOAD}, ~{SP_LO_OUT}, ~{SP_UP} -> Stack Pointer"
 		(exclude_from_sim no)
 		(at 161.798 170.434 0)
