File: dino_v0_0_2/input_output.kicad_sch (KiCad schematic)
At the start: 26 parts, among them SW1 SW_DIP_x08

Commit message: Dino v0.0.2 Schematic Update
Parts:
- renumbered SWITCH-GATE to SWITCH-GATE1
Other:
- title: Dino v0.0.1 -> Dino v0.0.2
Changed lines of the file:
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@@
 	(paper "USLetter")
 	(title_block
-		(title "Dino v0.0.1")
-		(date "2025-07-18")
+		(title "Dino v0.0.2")
+		(date "2025-07-19")
 		(rev "v1.0.4")
 		(comment 1 "Input Output Components")
@@
 		)
 		(instances
-			(project "dino_v0_0_1"
-				(path "/e43166a5-d972-471d-b3cf-9f4f12c7f541/746aad78-e591-4d08-b628-4d67d677e6d4"
+			(project "dino_v0_0_2"
+				(path "/e43166a5-d972-471d-b3cf-9f4f12c7f541/57977dc0-ee09-4ff5-b2e8-b5fa69d8270d"
 					(reference "#PWR06")
 					(unit 1)
@@
 		)
 		(instances
-			(project "dino_v0_0_1"
-				(path "/e43166a5-d972-471d-b3cf-9f4f12c7f541/746aad78-e591-4d08-b628-4d67d677e6d4"
+			(project "dino_v0_0_2"
+				(path "/e43166a5-d972-471d-b3cf-9f4f12c7f541/57977dc0-ee09-4ff5-b2e8-b5fa69d8270d"
 					(reference "D6")
 					(unit 1)
@@
 		)
 		(instances
-			(project "dino_v0_0_1"
-				(path "/e43166a5-d972-471d-b3cf-9f4f12c7f541/746aad78-e591-4d08-b628-4d67d677e6d4"
+			(project "dino_v0_0_2"
+				(path "/e43166a5-d972-471d-b3cf-9f4f12c7f541/57977dc0-ee09-4ff5-b2e8-b5fa69d8270d"
 					(reference "R10")
 					(unit 1)
@@
 		)
 		(instances
-			(project "dino_v0_0_1"
-				(path "/e43166a5-d972-471d-b3cf-9f4f12c7f541/746aad78-e591-4d08-b628-4d67d677e6d4"
+			(project "dino_v0_0_2"
+				(path "/e43166a5-d972-471d-b3cf-9f4f12c7f541/57977dc0-ee09-4ff5-b2e8-b5fa69d8270d"
 					(reference "R23")
 					(unit 1)
@@
 		)
 		(instances
-			(project "dino_v0_0_1"
-				(path "/e43166a5-d972-471d-b3cf-9f4f12c7f541/746aad78-e591-4d08-b628-4d67d677e6d4"
+			(project "dino_v0_0_2"
+				(path "/e43166a5-d972-471d-b3cf-9f4f12c7f541/57977dc0-ee09-4ff5-b2e8-b5fa69d8270d"
 					(reference "R19")
 					(unit 1)
@@
 		)
 		(instances
-			(project "dino_v0_0_1"
-				(path "/e43166a5-d972-471d-b3cf-9f4f12c7f541/746aad78-e591-4d08-b628-4d67d677e6d4"
+			(project "dino_v0_0_2"
+				(path "/e43166a5-d972-471d-b3cf-9f4f12c7f541/57977dc0-ee09-4ff5-b2e8-b5fa69d8270d"
 					(reference "R14")
 					(unit 1)
@@
 		)
 		(instances
-			(project "dino_v0_0_1"
-				(path "/e43166a5-d972-471d-b3cf-9f4f12c7f541/746aad78-e591-4d08-b628-4d67d677e6d4"
+			(project "dino_v0_0_2"
+				(path "/e43166a5-d972-471d-b3cf-9f4f12c7f541/57977dc0-ee09-4ff5-b2e8-b5fa69d8270d"
 					(reference "R21")
 					(unit 1)
@@
 		)
 		(instances
-			(project "dino_v0_0_1"
-				(path "/e43166a5-d972-471d-b3cf-9f4f12c7f541/746aad78-e591-4d08-b628-4d67d677e6d4"
+			(project "dino_v0_0_2"
+				(path "/e43166a5-d972-471d-b3cf-9f4f12c7f541/57977dc0-ee09-4ff5-b2e8-b5fa69d8270d"
 					(reference "R13")
 					(unit 1)
@@
 		)
 		(instances
-			(project "dino_v0_0_1"
-				(path "/e43166a5-d972-471d-b3cf-9f4f12c7f541/746aad78-e591-4d08-b628-4d67d677e6d4"
+			(project "dino_v0_0_2"
+				(path "/e43166a5-d972-471d-b3cf-9f4f12c7f541/57977dc0-ee09-4ff5-b2e8-b5fa69d8270d"
 					(reference "D4")
 					(unit 1)
@@
 		)
 		(instances
-			(project ""
-				(path "/e43166a5-d972-471d-b3cf-9f4f12c7f541/746aad78-e591-4d08-b628-4d67d677e6d4"
+			(project "dino_v0_0_2"
+				(path "/e43166a5-d972-471d-b3cf-9f4f12c7f541/57977dc0-ee09-4ff5-b2e8-b5fa69d8270d"
 					(reference "R9")
 					(unit 1)
@@
 		)
 		(instances
-			(project "dino_v0_0_1"
-				(path "/e43166a5-d972-471d-b3cf-9f4f12c7f541/746aad78-e591-4d08-b628-4d67d677e6d4"
+			(project "dino_v0_0_2"
+				(path "/e43166a5-d972-471d-b3cf-9f4f12c7f541/57977dc0-ee09-4ff5-b2e8-b5fa69d8270d"
 					(reference "D1")
 					(unit 1)
@@
 		)
 		(instances
-			(project "dino_v0_0_1"
-				(path "/e43166a5-d972-471d-b3cf-9f4f12c7f541/746aad78-e591-4d08-b628-4d67d677e6d4"
+			(project "dino_v0_0_2"
+				(path "/e43166a5-d972-471d-b3cf-9f4f12c7f541/57977dc0-ee09-4ff5-b2e8-b5fa69d8270d"
 					(reference "D3")
 					(unit 1)
@@
 		)
 		(instances
-			(project "dino_v0_0_1"
-				(path "/e43166a5-d972-471d-b3cf-9f4f12c7f541/746aad78-e591-4d08-b628-4d67d677e6d4"
+			(project "dino_v0_0_2"
+				(path "/e43166a5-d972-471d-b3cf-9f4f12c7f541/57977dc0-ee09-4ff5-b2e8-b5fa69d8270d"
 					(reference "D5")
 					(unit 1)
@@
 		)
 		(instances
-			(project "dino_v0_0_1"
-				(path "/e43166a5-d972-471d-b3cf-9f4f12c7f541/746aad78-e591-4d08-b628-4d67d677e6d4"
+			(project "dino_v0_0_2"
+				(path "/e43166a5-d972-471d-b3cf-9f4f12c7f541/57977dc0-ee09-4ff5-b2e8-b5fa69d8270d"
 					(reference "R24")
 					(unit 1)
@@
 		)
 		(instances
-			(project "dino_v0_0_1"
-				(path "/e43166a5-d972-471d-b3cf-9f4f12c7f541/746aad78-e591-4d08-b628-4d67d677e6d4"
+			(project "dino_v0_0_2"
+				(path "/e43166a5-d972-471d-b3cf-9f4f12c7f541/57977dc0-ee09-4ff5-b2e8-b5fa69d8270d"
 					(reference "D7")
 					(unit 1)
@@
 		)
 		(instances
-			(project "dino_v0_0_1"
-				(path "/e43166a5-d972-471d-b3cf-9f4f12c7f541/746aad78-e591-4d08-b628-4d67d677e6d4"
+			(project "dino_v0_0_2"
+				(path "/e43166a5-d972-471d-b3cf-9f4f12c7f541/57977dc0-ee09-4ff5-b2e8-b5fa69d8270d"
 					(reference "D8")
 					(unit 1)
@@
 		)
 		(instances
-			(project "dino_v0_0_1"
-				(path "/e43166a5-d972-471d-b3cf-9f4f12c7f541/746aad78-e591-4d08-b628-4d67d677e6d4"
+			(project "dino_v0_0_2"
+				(path "/e43166a5-d972-471d-b3cf-9f4f12c7f541/57977dc0-ee09-4ff5-b2e8-b5fa69d8270d"
 					(reference "R20")
 					(unit 1)
@@
 		)
 		(instances
-			(project "dino_v0_0_1"
-				(path "/e43166a5-d972-471d-b3cf-9f4f12c7f541/746aad78-e591-4d08-b628-4d67d677e6d4"
+			(project "dino_v0_0_2"
+				(path "/e43166a5-d972-471d-b3cf-9f4f12c7f541/57977dc0-ee09-4ff5-b2e8-b5fa69d8270d"
 					(reference "R15")
 					(unit 1)
@@
 		)
 		(instances
-			(project "dino_v0_0_1"
-				(path "/e43166a5-d972-471d-b3cf-9f4f12c7f541/746aad78-e591-4d08-b628-4d67d677e6d4"
+			(project "dino_v0_0_2"
+				(path "/e43166a5-d972-471d-b3cf-9f4f12c7f541/57977dc0-ee09-4ff5-b2e8-b5fa69d8270d"
 					(reference "R18")
 					(unit 1)
@@
 		)
 		(instances
-			(project "dino_v0_0_1"
-				(path "/e43166a5-d972-471d-b3cf-9f4f12c7f541/746aad78-e591-4d08-b628-4d67d677e6d4"
+			(project "dino_v0_0_2"
+				(path "/e43166a5-d972-471d-b3cf-9f4f12c7f541/57977dc0-ee09-4ff5-b2e8-b5fa69d8270d"
 					(reference "R16")
 					(unit 1)
@@
 		)
 		(instances
-			(project "dino_v0_0_1"
-				(path "/e43166a5-d972-471d-b3cf-9f4f12c7f541/746aad78-e591-4d08-b628-4d67d677e6d4"
+			(project "dino_v0_0_2"
+				(path "/e43166a5-d972-471d-b3cf-9f4f12c7f541/57977dc0-ee09-4ff5-b2e8-b5fa69d8270d"
 					(reference "R12")
 					(unit 1)
@@
 		)
 		(instances
-			(project "dino_v0_0_1"
-				(path "/e43166a5-d972-471d-b3cf-9f4f12c7f541/746aad78-e591-4d08-b628-4d67d677e6d4"
+			(project "dino_v0_0_2"
+				(path "/e43166a5-d972-471d-b3cf-9f4f12c7f541/57977dc0-ee09-4ff5-b2e8-b5fa69d8270d"
 					(reference "R11")
 					(unit 1)
@@
 		)
 		(instances
-			(project "dino_v0_0_1"
-				(path "/e43166a5-d972-471d-b3cf-9f4f12c7f541/746aad78-e591-4d08-b628-4d67d677e6d4"
+			(project "dino_v0_0_2"
+				(path "/e43166a5-d972-471d-b3cf-9f4f12c7f541/57977dc0-ee09-4ff5-b2e8-b5fa69d8270d"
 					(reference "#PWR04")
 					(unit 1)
@@
 		)
 		(instances
-			(project "dino_v0_0_1"
-				(path "/e43166a5-d972-471d-b3cf-9f4f12c7f541/746aad78-e591-4d08-b628-4d67d677e6d4"
+			(project "dino_v0_0_2"
+				(path "/e43166a5-d972-471d-b3cf-9f4f12c7f541/57977dc0-ee09-4ff5-b2e8-b5fa69d8270d"
 					(reference "R22")
 					(unit 1)
@@
 		)
 		(instances
-			(project ""
-				(path "/e43166a5-d972-471d-b3cf-9f4f12c7f541/746aad78-e591-4d08-b628-4d67d677e6d4"
+			(project "dino_v0_0_2"
+				(path "/e43166a5-d972-471d-b3cf-9f4f12c7f541/57977dc0-ee09-4ff5-b2e8-b5fa69d8270d"
 					(reference "SW1")
 					(unit 1)
@@
 		)
 		(instances
-			(project "dino_v0_0_1"
-				(path "/e43166a5-d972-471d-b3cf-9f4f12c7f541/746aad78-e591-4d08-b628-4d67d677e6d4"
+			(project "dino_v0_0_2"
+				(path "/e43166a5-d972-471d-b3cf-9f4f12c7f541/57977dc0-ee09-4ff5-b2e8-b5fa69d8270d"
 					(reference "R17")
 					(unit 1)
@@
 		(dnp no)
 		(fields_autoplaced yes)
-		(property "Reference" "SWITCH-GATE"
+		(property "Reference" "SWITCH-GATE1"
 			(at 92.3133 33.02 0)
 			(effects
@@
 		)
 		(instances
-			(project ""
-				(path "/e43166a5-d972-471d-b3cf-9f4f12c7f541/746aad78-e591-4d08-b628-4d67d677e6d4"
-					(reference "SWITCH-GATE")
+			(project "dino_v0_0_2"
+				(path "/e43166a5-d972-471d-b3cf-9f4f12c7f541/57977dc0-ee09-4ff5-b2e8-b5fa69d8270d"
+					(reference "SWITCH-GATE1")
 					(unit 1)
 				)
@@
 		)
 		(instances
-			(project "dino_v0_0_1"
-				(path "/e43166a5-d972-471d-b3cf-9f4f12c7f541/746aad78-e591-4d08-b628-4d67d677e6d4"
+			(project "dino_v0_0_2"
+				(path "/e43166a5-d972-471d-b3cf-9f4f12c7f541/57977dc0-ee09-4ff5-b2e8-b5fa69d8270d"
 					(reference "D2")
 					(unit 1)

Commit message: DINO Updates
Parts:
- added Bus-Arbiter1: 74LS645, symbol 74xx:74LS645
- added MCM60256AP1: SRAM, symbol Memory_RAM:MCM60256AP
Changed lines of the file:
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@@
 	(title_block
 		(title "Dino v0.0.2")
-		(date "2025-07-24")
-		(rev "v1.0.5")
+		(date "2025-07-28")
+		(rev "v1.0.7")
 		(comment 1 "Input Output Components")
 		(comment 3 "An 8-bit computer with 16-bit addressing and 16-bit control words")
@@
 	)
 	(symbol
+		(lib_id "74xx:74LS645")
+		(at 229.87 50.8 0)
+		(unit 1)
+		(exclude_from_sim no)
+		(in_bom yes)
+		(on_board yes)
+		(dnp no)
+		(property "Reference" "Bus-Arbiter1"
+			(at 232.41 31.242 0)
+			(effects
+				(font
+					(size 1.27 1.27)
+				)
+				(justify left)
+			)
+		)
+		(property "Value" "74LS645"
+			(at 232.41 33.782 0)
+			(effects
+				(font
+					(size 1.27 1.27)
+				)
+				(justify left)
+			)
+		)
+		(property "Footprint" ""
+			(at 229.87 50.8 0)
+			(effects
+				(font
+					(size 1.27 1.27)
+				)
+				(hide yes)
+			)
+		)
+		(property "Datasheet" ""
+			(at 229.87 50.8 0)
+			(effects
+				(font
+					(size 1.27 1.27)
+				)
+				(hide yes)
+			)
+		)
+		(property "Description" ""
+			(at 229.87 50.8 0)
+			(effects
+				(font
+					(size 1.27 1.27)
+				)
+				(hide yes)
+			)
+		)
+		(pin "5"
+		)
+		(pin "6"
+		)
+		(pin "1"
+		)
+		(pin "15"
+		)
+		(pin "14"
+		)
+		(pin "13"
+		)
+		(pin "12"
+		)
+		(pin "11"
+		)
+		(pin "19"
+		)
+		(pin "20"
+		)
+		(pin "10"
+		)
+		(pin "18"
+		)
+		(pin "17"
+		)
+		(pin "16"
+		)
+		(pin "3"
+		)
+		(pin "8"
+		)
+		(pin "2"
+		)
+		(pin "4"
+		)
+		(pin "7"
+		)
+		(pin "9"
+		)
+		(instances
+			(project "dino_v0_0_2"
+				(path "/e43166a5-d972-471d-b3cf-9f4f12c7f541/57977dc0-ee09-4ff5-b2e8-b5fa69d8270d"
+					(reference "Bus-Arbiter1")
+					(unit 1)
+				)
+			)
+		)
+	)
+	(symbol
 		(lib_id "Device:R")
 		(at 125.73 76.2 90)
@@
 					(unit 1)
 				)
+			)
+		)
+	)
+	(symbol
+		(lib_id "Memory_RAM:MCM60256AP")
+		(at 194.31 83.82 0)
+		(unit 1)
+		(exclude_from_sim no)
+		(in_bom yes)
+		(on_board yes)
+		(dnp no)
+		(property "Reference" "MCM60256AP1"
+			(at 198.374 103.378 90)
+			(effects
+				(font
+					(size 1.27 1.27)
+					(thickness 0.1588)
+				)
+				(justify left)
+			)
+		)
+		(property "Value" "SRAM"
+			(at 196.342 100.076 90)
+			(effects
+				(font
+					(size 1.27 1.27)
+					(thickness 0.254)
+					(bold yes)
+					(color 194 0 194 1)
+				)
+				(justify left)
+			)
+		)
+		(property "Footprint" ""
+			(at 194.31 83.82 0)
+			(effects
+				(font
+					(size 1.27 1.27)
+				)
+				(hide yes)
+			)
+		)
+		(property "Datasheet" ""
+			(at 194.31 83.82 0)
+			(effects
+				(font
+					(size 1.27 1.27)
+				)
+				(hide yes)
+			)
+		)
+		(property "Description" ""
+			(at 194.31 83.82 0)
+			(effects
+				(font
+					(size 1.27 1.27)
+				)
+				(hide yes)
+			)
+		)
+		(pin "5"
+		)
+		(pin "4"
+		)
+		(pin "8"
+		)
+		(pin "7"
+		)
+		(pin "6"
+		)
+		(pin "10"
+		)
+		(pin "9"
+		)
+		(pin "17"
+		)
+		(pin "18"
+		)
+		(pin "19"
+		)
+		(pin "3"
+		)
+		(pin "25"
+		)
+		(pin "24"
+		)
+		(pin "21"
+		)
+		(pin "23"
+		)
+		(pin "2"
+		)
+		(pin "26"
+		)
+		(pin "1"
+		)
+		(pin "27"
+		)
+		(pin "22"
+		)
+		(pin "28"
+		)
+		(pin "20"
+		)
+		(pin "14"
+		)
+		(pin "11"
+		)
+		(pin "12"
+		)
+		(pin "13"
+		)
+		(pin "15"
+		)
+		(pin "16"
+		)
+		(instances
+			(project "dino_v0_0_2"
+				(path "/e43166a5-d972-471d-b3cf-9f4f12c7f541/57977dc0-ee09-4ff5-b2e8-b5fa69d8270d"
+					(reference "MCM60256AP1")
+					(unit 1)
+				)

Commit message: Update
Parts:
- removed Bus-Arbiter1: 74LS645, symbol 74xx:74LS645
- removed MCM60256AP1: SRAM, symbol Memory_RAM:MCM60256AP
Changed lines of the file:
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@@
-	)
-	(symbol
-		(lib_id "74xx:74LS645")
-		(at 229.87 50.8 0)
-		(unit 1)
-		(exclude_from_sim no)
-		(in_bom yes)
-		(on_board yes)
-		(dnp no)
-		(property "Reference" "Bus-Arbiter1"
-			(at 232.41 31.242 0)
-			(effects
-				(font
-					(size 1.27 1.27)
-				)
-				(justify left)
-			)
-		)
-		(property "Value" "74LS645"
-			(at 232.41 33.782 0)
-			(effects
-				(font
-					(size 1.27 1.27)
-				)
-				(justify left)
-			)
-		)
-		(property "Footprint" ""
-			(at 229.87 50.8 0)
-			(effects
-				(font
-					(size 1.27 1.27)
-				)
-				(hide yes)
-			)
-		)
-		(property "Datasheet" ""
-			(at 229.87 50.8 0)
-			(effects
-				(font
-					(size 1.27 1.27)
-				)
-				(hide yes)
-			)
-		)
-		(property "Description" ""
-			(at 229.87 50.8 0)
-			(effects
-				(font
-					(size 1.27 1.27)
-				)
-				(hide yes)
-			)
-		)
-		(pin "5"
-		)
-		(pin "6"
-		)
-		(pin "1"
-		)
-		(pin "15"
-		)
-		(pin "14"
-		)
-		(pin "13"
-		)
-		(pin "12"
-		)
-		(pin "11"
-		)
-		(pin "19"
-		)
-		(pin "20"
-		)
-		(pin "10"
-		)
-		(pin "18"
-		)
-		(pin "17"
-		)
-		(pin "16"
-		)
-		(pin "3"
-		)
-		(pin "8"
-		)
-		(pin "2"
-		)
-		(pin "4"
-		)
-		(pin "7"
-		)
-		(pin "9"
-		)
-		(instances
-			(project "dino_v0_0_2"
-				(path "/e43166a5-d972-471d-b3cf-9f4f12c7f541/57977dc0-ee09-4ff5-b2e8-b5fa69d8270d"
-					(reference "Bus-Arbiter1")
-					(unit 1)
-				)
-			)
-		)
 	)
 	(symbol
@@
 					(unit 1)
 				)
-			)
-		)
-	)
-	(symbol
-		(lib_id "Memory_RAM:MCM60256AP")
-		(at 194.31 83.82 0)
-		(unit 1)
-		(exclude_from_sim no)
-		(in_bom yes)
-		(on_board yes)
-		(dnp no)
-		(property "Reference" "MCM60256AP1"
-			(at 198.374 103.378 90)
-			(effects
-				(font
-					(size 1.27 1.27)
-					(thickness 0.1588)
-				)
-				(justify left)
-			)
-		)
-		(property "Value" "SRAM"
-			(at 196.342 100.076 90)
-			(effects
-				(font
-					(size 1.27 1.27)
-					(thickness 0.254)
-					(bold yes)
-					(color 194 0 194 1)
-				)
-				(justify left)
-			)
-		)
-		(property "Footprint" ""
-			(at 194.31 83.82 0)
-			(effects
-				(font
-					(size 1.27 1.27)
-				)
-				(hide yes)
-			)
-		)
-		(property "Datasheet" ""
-			(at 194.31 83.82 0)
-			(effects
-				(font
-					(size 1.27 1.27)
-				)
-				(hide yes)
-			)
-		)
-		(property "Description" ""
-			(at 194.31 83.82 0)
-			(effects
-				(font
-					(size 1.27 1.27)
-				)
-				(hide yes)
-			)
-		)
-		(pin "5"
-		)
-		(pin "4"
-		)
-		(pin "8"
-		)
-		(pin "7"
-		)
-		(pin "6"
-		)
-		(pin "10"
-		)
-		(pin "9"
-		)
-		(pin "17"
-		)
-		(pin "18"
-		)
-		(pin "19"
-		)
-		(pin "3"
-		)
-		(pin "25"
-		)
-		(pin "24"
-		)
-		(pin "21"
-		)
-		(pin "23"
-		)
-		(pin "2"
-		)
-		(pin "26"
-		)
-		(pin "1"
-		)
-		(pin "27"
-		)
-		(pin "22"
-		)
-		(pin "28"
-		)
-		(pin "20"
-		)
-		(pin "14"
-		)
-		(pin "11"
-		)
-		(pin "12"
-		)
-		(pin "13"
-		)
-		(pin "15"
-		)
-		(pin "16"
-		)
-		(instances
-			(project "dino_v0_0_2"
-				(path "/e43166a5-d972-471d-b3cf-9f4f12c7f541/57977dc0-ee09-4ff5-b2e8-b5fa69d8270d"
-					(reference "MCM60256AP1")
-					(unit 1)
-				)
