File: dino_v0_0_2/input_output.kicad_sch (KiCad schematic)
At the start: 24 parts

Commit message: feat(kicad): footprints, power sheet, global labels, PCB draft
Every symbol gets a stock THT footprint (plain DIP, no sockets, so the
3D render shows ICs). New Power sheet: 24-pin ATX header for a picoPSU,
rails +5V/+3.3V/+12V/-12V/GND only; no -5V exists on any ATX unit since
2003, none drawn. PS_ON# on a 2-pin header.

Cross-sheet labels become global labels. KiCad joined nothing between
sheets before: 122 base names were split per sheet, ERC saw 90 undriven
inputs whose driver sat one sheet away, and the PCB ratsnest stopped at
every sheet boundary. Proof: KiCad's netlist after equals a name-join of
its netlist before plus the 15 CW alias pairs, pin for pin.

kicad_contracts took a node's sheet from the net name's /Sheet/ prefix;
global nets have none, so it emitted an empty contracts doc. Sheet now
comes from the component's own path; the doc regenerates with zero diff.

ERC 477 -> 2. Real fixes: ROM I/O pins input -> tri_state, '382 GND pin
power_out -> power_in, four orphan symbols rehomed to project lib `dino`,
one stub wire. 133 by-design warnings excluded by uuid ('245 readback on
counter Q, alias stubs, probe-point labels); the two left are bus
signals the peripheral bus sheet will consume.

PCB draft: 198 footprints placed per sheet, all pads netted, no tracks.

Co-Authored-By: Claude Fable 5.1 <noreply@anthropic.com>
Claude-Session: https://claude.ai/code/session_018irreFHb1xEykW5kCD26ow
Parts:
- D1, D2, D3, D4, D5, D6, D7, D8: footprint (none) -> LED_THT:LED_D5.0mm
- R10, R11, R12, R13, R14, R15, R16, R25, R26, R27, R4, R5, R6, R7, R8, R9: footprint (none) -> Resistor_THT:R_Axial_DIN0207_L6.3mm_D2.5mm_P10.16mm_Horizontal
