File: dino_v0_0_2/microcode.kicad_sch (KiCad schematic)
At the start: 4 parts, among them U15 AT28C64B, U16 74LS244N, U17 74LS244N, U9 AT28C64B

Commit message: Update
Other:
- moved on the sheet: U15, U16, U17, U9

Commit message: Schematics WIP
Changed lines of the file:
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@@
 		)
 	)
-	(label "Instruction Register"
+	(label "Instruction Register Bus"
 		(at 69.85 52.07 180)
 		(effects

Commit message: Schematic Update
Connections:
- net +5V: now also U17.19 (2~{G}); no longer U16.19 (2~{G})
- net GND: now also U16.19 (2~{G}); no longer U17.19 (2~{G})
- net at U15.21 (A10), U9.21 (A10): now also U16.5 (2Y3); no longer U16.14 (1Y3)
- net at U15.23 (A11), U9.23 (A11): now also U16.3 (2Y4); no longer U16.12 (1Y4)
- net at U15.24 (A9), U9.24 (A9): now also U16.7 (2Y2); no longer U16.16 (1Y2)
- net at U15.25 (A8), U9.25 (A8): now also U16.9 (2Y1); no longer U16.18 (1Y1)
- net at U15.3 (A7), U9.3 (A7): now also U16.12 (1Y4); no longer U17.3 (2Y4)
- net at U15.4 (A6), U9.4 (A6): now also U16.14 (1Y3); no longer U17.5 (2Y3)
- net at U15.5 (A5), U9.5 (A5): now also U16.16 (1Y2); no longer U17.7 (2Y2)
- net at U15.6 (A4), U9.6 (A4): now also U16.18 (1Y1); no longer U17.9 (2Y1)
