File: dino_v0_0_2/memory.kicad_sch (KiCad schematic)
At the start: 6 parts, among them U19 74LS244N, U20 74LS02, U21 74LS245, U24 AT28C256, U26 MCM60256AP, U40 74LS121

Commit message: Schematic Update
Parts:
- removed U19: 74LS244N, symbol 74xx:74LS244N
- added U19: 74LS245, symbol 74xx:74LS245
Connections:
- net +5V: now also U24.27 (~{WE}), U19.20 (VCC)
- net GND: now also U19.1 (DIR), U19.10 (GND)
- net ~{ROM_OUT}: now also U19.19 (CE)
- net at U24.16 (I/O4): now also U19.14 (B4)
- net at U24.17 (I/O5): now also U19.13 (B5)
- net at U24.18 (I/O6): now also U19.12 (B6)
- net at U24.19 (I/O7): now also U19.11 (B7)
- net at U24.11 (I/O0): now also U19.18 (B0)
- net at U24.12 (I/O1): now also U19.17 (B1)
- net at U24.13 (I/O2): now also U19.16 (B2)
- net at U24.15 (I/O3): now also U19.15 (B3)
- no-connect marks 4 -> 3
Changed lines of the file:
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@@
 	)
 	(junction
-		(at 109.22 111.76)
+		(at 162.56 93.98)
 		(diameter 0)
 		(color 0 0 0 0)
 	)
 	(junction
-		(at 194.31 83.82)
+		(at 109.22 111.76)
 		(diameter 0)
 		(color 0 0 0 0)
@@
 	)
 	(junction
+		(at 167.64 91.44)
+		(diameter 0)
+		(color 0 0 0 0)
+	)
+	(junction
 		(at 166.37 127)
 		(diameter 0)
@@
 	)
 	(no_connect
-		(at 210.82 107.95)
-	)
-	(no_connect
 		(at 111.76 144.78)
 	)
@@
 	(wire
 		(pts
+			(xy 168.91 81.28) (xy 167.64 81.28)
+		)
+		(stroke
+			(width 0)
+			(type default)
+		)
+	)
+	(wire
+		(pts
 			(xy 102.87 152.4) (xy 102.87 146.05)
 		)
@@
 		)
 	)
+	(wire
+		(pts
+			(xy 162.56 93.98) (xy 162.56 96.52)
+		)
+		(stroke
+			(width 0)
+			(type default)
+		)
+	)
 	(bus
 		(pts
@@
 	(wire
 		(pts
+			(xy 167.64 81.28) (xy 167.64 91.44)
+		)
+		(stroke
+			(width 0)
+			(type default)
+		)
+	)
+	(wire
+		(pts
 			(xy 204.47 73.66) (xy 194.31 73.66)
 		)
@@
 		)
 	)
+	(wire
+		(pts
+			(xy 209.55 107.95) (xy 209.55 93.98)
+		)
+		(stroke
+			(width 0)
+			(type default)
+		)
+	)
 	(bus
 		(pts
@@
 		)
 	)
+	(wire
+		(pts
+			(xy 210.82 107.95) (xy 209.55 107.95)
+		)
+		(stroke
+			(width 0)
+			(type default)
+		)
+	)
 	(bus
 		(pts
@@
 	(wire
 		(pts
+			(xy 209.55 93.98) (xy 162.56 93.98)
+		)
+		(stroke
+			(width 0)
+			(type default)
+		)
+	)
+	(wire
+		(pts
 			(xy 134.62 60.96) (xy 148.59 60.96)
 		)
@@
 	(wire
 		(pts
-			(xy 162.56 40.64) (xy 162.56 96.52)
+			(xy 162.56 40.64) (xy 162.56 93.98)
 		)
 		(stroke
@@
 	(wire
 		(pts
-			(xy 194.31 83.82) (xy 194.31 111.76)
-		)
-		(stroke
-			(width 0)
-			(type default)
-		)
-	)
-	(wire
-		(pts
 			(xy 220.98 140.97) (xy 226.06 140.97)
 		)
@@
 	(wire
 		(pts
-			(xy 151.13 91.44) (xy 181.61 91.44)
+			(xy 151.13 91.44) (xy 167.64 91.44)
 		)
 		(stroke
@@
 		)
 	)
+	(wire
+		(pts
+			(xy 194.31 96.52) (xy 194.31 111.76)
+		)
+		(stroke
+			(width 0)
+			(type default)
+		)
+	)
 	(bus
 		(pts
@@
 	(wire
 		(pts
-			(xy 106.68 81.28) (xy 109.22 81.28)
+			(xy 168.91 83.82) (xy 168.91 96.52)
 		)
 		(stroke
@@
 	(wire
 		(pts
-			(xy 168.91 71.12) (xy 153.67 71.12)
+			(xy 106.68 81.28) (xy 109.22 81.28)
 		)
 		(stroke
@@
 		)
 	)
-	(bus
+	(wire
 		(pts
-			(xy 151.13 63.5) (xy 151.13 66.04)
+			(xy 168.91 71.12) (xy 153.67 71.12)
 		)
 		(stroke
@@
 		)
 	)
-	(wire
+	(bus
 		(pts
-			(xy 209.55 63.5) (xy 194.31 63.5)
+			(xy 151.13 63.5) (xy 151.13 66.04)
 		)
 		(stroke
@@
 	(wire
 		(pts
-			(xy 203.2 76.2) (xy 194.31 76.2)
+			(xy 209.55 63.5) (xy 194.31 63.5)
 		)
 		(stroke
@@
 	(wire
 		(pts
-			(xy 194.31 81.28) (xy 194.31 83.82)
+			(xy 203.2 76.2) (xy 194.31 76.2)
 		)
 		(stroke
@@
 	(wire
 		(pts
+			(xy 167.64 91.44) (xy 181.61 91.44)
+		)
+		(stroke
+			(width 0)
+			(type default)
+		)
+	)
+	(wire
+		(pts
 			(xy 134.62 66.04) (xy 148.59 66.04)
 		)
@@
 	(wire
 		(pts
+			(xy 168.91 96.52) (xy 194.31 96.52)
+		)
+		(stroke
+			(width 0)
+			(type default)
+		)
+	)
+	(wire
+		(pts
 			(xy 210.82 85.09) (xy 203.2 85.09)
 		)
@@
 	)
 	(symbol
-		(lib_id "74xx:74LS02")
-		(at 233.68 143.51 0)
+		(lib_id "74xx:74LS245")
+		(at 181.61 71.12 0)
 		(unit 1)
 		(exclude_from_sim no)
@@
 		(dnp no)
 		(fields_autoplaced yes)
-		(property "Reference" "U20"
-			(at 233.68 134.62 0)
+		(property "Reference" "U19"
+			(at 183.7533 50.8 0)
 			(effects
 				(font
 					(size 1.27 1.27)
 				)
+				(justify left)
 			)
 		)
-		(property "Value" "74LS02"
-			(at 233.68 137.16 0)
+		(property "Value" "74LS245"
+			(at 183.7533 53.34 0)
 			(effects
 				(font
 					(size 1.27 1.27)
 				)
+				(justify left)
 			)
 		)
 		(property "Footprint" ""
-			(at 233.68 143.51 0)
+			(at 181.61 71.12 0)
 			(effects
 				(font
@@
 			)
 		)
-		(property "Datasheet" "http://www.ti.com/lit/gpn/sn74ls02"
-			(at 233.68 143.51 0)
+		(property "Datasheet" "http://www.ti.com/lit/gpn/sn74LS245"
+			(at 181.61 71.12 0)
 			(effects
 				(font
@@
 			)
 		)
-		(property "Description" "quad 2-input NOR gate"
-			(at 233.68 143.51 0)
+		(property "Description" "Octal BUS Transceivers, 3-State outputs"
+			(at 181.61 71.12 0)
 			(effects
 				(font
@@
 			)
 		)
-		(pin "11"
+		(pin "19"
 		)
-		(pin "12"
+		(pin "20"
 		)
-		(pin "13"
+		(pin "10"
+		)
+		(pin "18"
+		)
+		(pin "17"
+		)
+		(pin "16"
+		)
+		(pin "15"
 		)
 		(pin "14"
 		)
-		(pin "7"
+		(pin "13"
+		)
+		(pin "12"
+		)
+		(pin "11"
 		)
 		(pin "2"
@@
 		(pin "3"
 		)
-		(pin "1"
+		(pin "4"
 		)
 		(pin "5"
@@
 		(pin "6"
 		)
-		(pin "4"
+		(pin "7"
 		)
 		(pin "8"
@@
 		(pin "9"
 		)
-		(pin "10"
+		(pin "1"
 		)
 		(instances
 			(project "dino_v0_0_2"
 				(path "/e43166a5-d972-471d-b3cf-9f4f12c7f541/b0594337-21bc-457d-8ae7-405a6ec1dde7"
-					(reference "U20")
+					(reference "U19")
 					(unit 1)
 				)
@@
 	)
 	(symbol
-		(lib_id "74xx:74LS244N")
-		(at 181.61 71.12 0)
-		(mirror y)
+		(lib_id "74xx:74LS02")
+		(at 233.68 143.51 0)
 		(unit 1)
 		(exclude_from_sim no)
@@
 		(dnp no)
 		(fields_autoplaced yes)
-		(property "Reference" "U19"
-			(at 179.4667 50.8 0)
+		(property "Reference" "U20"
+			(at 233.68 134.62 0)
 			(effects
 				(font
 					(size 1.27 1.27)
 				)
-				(justify left)
 			)
 		)
-		(property "Value" "74LS244N"
-			(at 179.4667 53.34 0)
+		(property "Value" "74LS02"
+			(at 233.68 137.16 0)
 			(effects
 				(font
 					(size 1.27 1.27)
 				)
-				(justify left)
 			)
 		)
 		(property "Footprint" ""
-			(at 181.61 71.12 0)
+			(at 233.68 143.51 0)
 			(effects
 				(font
@@
 			)
 		)
-		(property "Datasheet" "http://www.ti.com/lit/ds/symlink/sn74ls244.pdf"
-			(at 180.086 94.234 0)
+		(property "Datasheet" "http://www.ti.com/lit/gpn/sn74ls02"
+			(at 233.68 143.51 0)
 			(effects
 				(font
@@
 			)
 		)
-		(property "Description" "Octal Buffer and Line Driver With 3-State Output, active-low enables, non-inverting outputs"
-			(at 182.118 47.244 0)
+		(property "Description" "quad 2-input NOR gate"
+			(at 233.68 143.51 0)
 			(effects
 				(font
@@
 			)
 		)
-		(pin "2"
-		)
-		(pin "4"
-		)
-		(pin "6"
-		)
-		(pin "8"
-		)
 		(pin "11"
 		)
-		(pin "13"
+		(pin "12"
 		)
-		(pin "15"
+		(pin "13"
 		)
-		(pin "17"
+		(pin "14"
 		)
-		(pin "1"
+		(pin "7"
 		)
-		(pin "19"
+		(pin "2"
 		)
-		(pin "20"
+		(pin "3"
 		)
-		(pin "10"
+		(pin "1"
 		)
-		(pin "18"
+		(pin "5"
 		)
-		(pin "16"
+		(pin "6"
 		)
-		(pin "14"
+		(pin "4"
 		)
-		(pin "12"
+		(pin "8"
 		)
 		(pin "9"
 		)
-		(pin "7"
-		)
-		(pin "5"
-		)
-		(pin "3"
+		(pin "10"
 		)
 		(instances
 			(project "dino_v0_0_2"
 				(path "/e43166a5-d972-471d-b3cf-9f4f12c7f541/b0594337-21bc-457d-8ae7-405a6ec1dde7"
-					(reference "U19")
+					(reference "U20")
 					(unit 1)
 				)

Commit message: KiCAD Updates
- Updating Memory Module
Parts:
- added C15: 100pF, symbol Device:C_Small
- added R4: 2.2kΩ, symbol Device:R
- added U51: 7400, symbol 74xx:7400
Connections:
- net +5V: now also U19.1 (DIR), U40.5 (B), U51.14 (VCC); no longer U40.9 (Rint)
- net GND: now also R4.1, U51.7 (GND); no longer U19.1 (DIR)
- net PULSE_REQ: now also U51.2; no longer U40.5 (B)
- net RAM_LOAD: now also U51.1; no longer U20.8, U20.9
- net at U40.4 (A2): now also U51.3; no longer U20.10
- net at U19.11 (B7): no longer U24.19 (I/O7)
- net at U19.12 (B6): no longer U24.18 (I/O6)
- net at U19.13 (B5): no longer U24.17 (I/O5)
- net at U19.14 (B4): no longer U24.16 (I/O4)
- net at U19.15 (B3): no longer U24.15 (I/O3)
- net at U19.16 (B2): no longer U24.13 (I/O2)
- net at U19.17 (B1): no longer U24.12 (I/O1)
- net at U19.18 (B0): no longer U24.11 (I/O0)
- net at U19.2 (A0): now also U24.11 (I/O0)
- net at U19.3 (A1): now also U24.12 (I/O1)
- net at U19.4 (A2): now also U24.13 (I/O2)
- net at U19.5 (A3): now also U24.15 (I/O3)
- net at U19.6 (A4): now also U24.16 (I/O4)
- net at U19.7 (A5): now also U24.17 (I/O5)
- net at U19.8 (A6): now also U24.18 (I/O6)
- net at U19.9 (A7): now also U24.19 (I/O7)
- net at U40.10 (Cext): now also C15.2
- net at U40.11 (R/Cext): now also C15.1, R4.2
- no-connect marks 3 -> 14
Other:
- moved on the sheet: U20B, U20C, U20D
