File: dino_v0_0_2/memory.kicad_sch (KiCad schematic)
At the start: 9 parts, among them U19 74LS245, U20 74LS02, U21 74LS245, U24 AT28C256, U26 MCM60256AP, U40 74LS121, U51 7400

Commit message: v0.3.0 - Rev 1.2.0 Update
Parts:
- removed C15: 100pF, symbol Device:C_Small
- removed R4: 2.2kΩ, symbol Device:R
- removed U20: 74LS02, symbol 74xx:74LS02
- removed U40: 74LS121, symbol 74xx:74LS121
Connections:
- net PULSE_REQ is gone; now on net WRITE_DIR: U51.2
- net RAM_LOAD is gone; now on net WRITE_DIR: U51.1
- net RAM_OUT is gone; now on net ~{WRITE_DIR}: U21.1 (DIR)
- net ~{RAM_LOAD} is gone; now on net ~{RAM_WRITE_EN}: U26.27 (~{WE})
- net ~{WRITE_DIR}: now reaches U51.3
- net ~{CLK}: now reaches U51.4
- net WRITE_DIR: now reaches U51.5
- net ~{RAM_WRITE_EN}: now reaches U51.6
- net ~{ROM_OUT}: no longer names the net of U19.19 (CE), U24.22 (~{OE})
- net ~{ROM_OUT}: no longer U24.20 (~{CE})
- new net ROM_EN: U24.20 (~{CE})
- no-connect marks 14 -> 7
Other:
- note added: "Defined on MAR"
- note added: "Derived from INV(A15) from MAR"
- note added: "ROM 0x0000-0x7FFF, RAM 0x8000-0xFFFF, selected by A15"
- note added: "WRITE_DIR net is defined on MDR"
- title: Dino v0.0.2 -> Dino v0.0.3
- moved on the sheet: U51A, U51B
