File: dino_v0_0_2/dino_v0_0_2.kicad_sch (KiCad schematic)
At the start: 13 parts, among them U5 7400, U6 74LS163, U7 74LS138, U8 74LS138

Commit message: Schematic Updates
Other:
- sheet Register Modules renamed Register Modules ( A + B )
- added sheet ALU Module (alu.kicad_sch)
- added sheet Register Modules ( C + Out ) (registers_c_out.kicad_sch)
- sheet Register Modules ( A + B ): file registers.kicad_sch -> registers_a_b.kicad_sch
Changed lines of the file:
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@@
+	)
+	(sheet
+		(at 237.49 68.58)
+		(size 12.7 11.43)
+		(exclude_from_sim no)
+		(in_bom yes)
+		(on_board yes)
+		(dnp no)
+		(fields_autoplaced yes)
+		(stroke
+			(width 0.1524)
+			(type solid)
+		)
+		(fill
+			(color 0 0 0 0.0000)
+		)
+		(property "Sheetname" "Register Modules ( C + Out )"
+			(at 237.49 67.8684 0)
+			(effects
+				(font
+					(size 1.27 1.27)
+				)
+				(justify left bottom)
+			)
+		)
+		(property "Sheetfile" "registers_c_out.kicad_sch"
+			(at 237.49 80.5946 0)
+			(effects
+				(font
+					(size 1.27 1.27)
+				)
+				(justify left top)
+			)
+		)
+		(instances
+			(project "dino_v0_0_2"
+				(path "/e43166a5-d972-471d-b3cf-9f4f12c7f541"
+					(page "8")
+				)
+			)
+		)
 	)
 	(sheet
@@
 			(project "dino_v0_0_2"
 				(path "/e43166a5-d972-471d-b3cf-9f4f12c7f541"
-					(page "8")
+					(page "10")
 				)
 			)
@@
 	)
 	(sheet
+		(at 217.805 67.945)
+		(size 12.7 11.43)
+		(exclude_from_sim no)
+		(in_bom yes)
+		(on_board yes)
+		(dnp no)
+		(fields_autoplaced yes)
+		(stroke
+			(width 0.1524)
+			(type solid)
+		)
+		(fill
+			(color 0 0 0 0.0000)
+		)
+		(property "Sheetname" "ALU Module"
+			(at 217.805 67.2334 0)
+			(effects
+				(font
+					(size 1.27 1.27)
+				)
+				(justify left bottom)
+			)
+		)
+		(property "Sheetfile" "alu.kicad_sch"
+			(at 217.805 79.9596 0)
+			(effects
+				(font
+					(size 1.27 1.27)
+				)
+				(justify left top)
+			)
+		)
+		(instances
+			(project "dino_v0_0_2"
+				(path "/e43166a5-d972-471d-b3cf-9f4f12c7f541"
+					(page "9")
+				)
+			)
+		)
+	)
+	(sheet
 		(at 160.02 45.72)
 		(size 12.7 12.7)
@@
 			(color 0 0 0 0.0000)
 		)
-		(property "Sheetname" "Register Modules"
+		(property "Sheetname" "Register Modules ( A + B )"
 			(at 187.96 66.5984 0)
 			(effects
@@
 			)
 		)
-		(property "Sheetfile" "registers.kicad_sch"
+		(property "Sheetfile" "registers_a_b.kicad_sch"
 			(at 187.96 79.3246 0)
 			(effects

Commit message: Separate Registers from Trigger Logic
Other:
- sheet Register Modules ( A + B ) renamed Register Modules
- removed sheet Register Modules ( C + Out )
- added sheet Register Logic (reg_logic.kicad_sch)
Changed lines of the file:
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@@
 	)
 	(sheet
-		(at 237.49 68.58)
+		(at 224.155 47.625)
 		(size 12.7 11.43)
 		(exclude_from_sim no)
@@
 			(color 0 0 0 0.0000)
 		)
-		(property "Sheetname" "Register Modules ( C + Out )"
-			(at 237.49 67.8684 0)
-			(effects
-				(font
-					(size 1.27 1.27)
-				)
-				(justify left bottom)
-			)
-		)
-		(property "Sheetfile" "registers_c_out.kicad_sch"
-			(at 237.49 80.5946 0)
-			(effects
-				(font
-					(size 1.27 1.27)
-				)
-				(justify left top)
-			)
-		)
-		(instances
-			(project "dino_v0_0_2"
-				(path "/e43166a5-d972-471d-b3cf-9f4f12c7f541"
-					(page "8")
+		(property "Sheetname" "Register Logic"
+			(at 224.155 46.9134 0)
+			(effects
+				(font
+					(size 1.27 1.27)
+				)
+				(justify left bottom)
+			)
+		)
+		(property "Sheetfile" "reg_logic.kicad_sch"
+			(at 224.155 59.6396 0)
+			(effects
+				(font
+					(size 1.27 1.27)
+				)
+				(justify left top)
+			)
+		)
+		(instances
+			(project "dino_v0_0_2"
+				(path "/e43166a5-d972-471d-b3cf-9f4f12c7f541"
+					(page "7")
 				)
 			)
@@
 	)
 	(sheet
-		(at 217.805 67.945)
+		(at 186.69 67.31)
 		(size 12.7 11.43)
 		(exclude_from_sim no)
@@
 		)
 		(property "Sheetname" "ALU Module"
-			(at 217.805 67.2334 0)
+			(at 186.69 66.5984 0)
 			(effects
 				(font
@@
 		)
 		(property "Sheetfile" "alu.kicad_sch"
-			(at 217.805 79.9596 0)
+			(at 186.69 79.3246 0)
 			(effects
 				(font
@@
 	)
 	(sheet
-		(at 187.96 67.31)
+		(at 208.28 67.945)
 		(size 12.7 11.43)
 		(exclude_from_sim no)
@@
 			(color 0 0 0 0.0000)
 		)
-		(property "Sheetname" "Register Modules ( A + B )"
-			(at 187.96 66.5984 0)
+		(property "Sheetname" "Register Modules"
+			(at 208.28 67.2334 0)
 			(effects
 				(font
@@
 		)
 		(property "Sheetfile" "registers_a_b.kicad_sch"
-			(at 187.96 79.3246 0)
-			(effects
-				(font
-					(size 1.27 1.27)
-				)
-				(justify left top)
-			)
-		)
-		(instances
-			(project "dino_v0_0_2"
-				(path "/e43166a5-d972-471d-b3cf-9f4f12c7f541"
-					(page "7")
-				)
-			)
+			(at 208.28 79.9596 0)
+			(effects
+				(font
+					(size 1.27 1.27)
+				)
+				(justify left top)
+			)
+		)
+		(instances
+			(project "dino_v0_0_2"
+				(path "/e43166a5-d972-471d-b3cf-9f4f12c7f541"
+					(page "8")
+				)
+			)
