File: dino_v0_0_2/dino_v0_0_2.kicad_sch (KiCad schematic)
At the start: 13 parts, among them U5 7400, U6 74LS163, U7 74LS138, U8 74LS138

Commit message: v0.3.0 - Rev 1.2.0 Update
Parts:
- removed U5: 7400, symbol 74xx:7400
- added U23: 74LS04, symbol 74xx:74LS04
Connections:
- net +5V: now also U23.14 (VCC)
- net CLK: now also U23.4; no longer SystemTimer.3 (Q)
- net GND: now also U23.7 (GND)
- net at U7.6 (E3): now also U23.6
- net at U6.11 (Q3), U8.6 (E3): now also U23.5
- new net SRC_CLK: SystemTimer.3 (Q), U23.1
- new net ~{CLK}: U23.2, U23.3
- no-connect marks 10 -> 7
Other:
- removed sheet Register Logic
- title: Dino v0.0.2 -> Dino v0.0.3
