File: dino_v0_0_2/dino_v0_0_2.kicad_sch (KiCad schematic)
At the start: 18 parts, among them SW2 RESET_BTN, U20 74LS163, U27 74LS74, U56 74HC14, U6 74LS163, U61 74LS02, U7 74LS138, U8 74LS138, Y1 4MHz

Commit message: Stack pointer + third microcode EEPROM: schematic, tooling, and ISA
Twelve chips, four sheets, seven instructions. The whole stack executes on
the gate model; the rig is detached so nothing has run on real hardware.

  U23         AT28C64B   third microcode EEPROM, CW16-23     microcode
  U70 / U71   '138       SRC / DST bank-1 decoders           control_word
  U63-U66     '169       16-bit stack pointer                stack_pointer
  U67 / U68   '245       SP hi/lo readback -> MDR            stack_pointer
  U69         '08        ~{SP_CE} = AND(~SP_UP, ~SP_DOWN)    stack_pointer
  U72 / U73   '245       PC0-7 / PC8-15 -> MDR               mdr

  LXISP 0x14   CALL 0x33   RET 0x34
  PUSHA 0x61   POPA 0x62   PUSHB 0x63   POPB 0x64

THE CONTROL WORD IS 24 BITS. Every new bit is polarised so 0xFF -- an erased
AT28C64B -- is today's machine, the same reasoning that made HALT=0xFF. Only
~{SRC_BANK} and ~{DST_BANK} are wired; ~{CIN_SEL}, ~{MISC_BANK},
~{ADDR_SEL1}, FLAG_SEL0/1 and FLAG_POL are burned into all 4096 rows and
wired to nothing, so no reburn is needed when their decode arrives.

Bank switching costs zero inverters: E3 is active-high and E1 active-low, so
bank 0 hangs off E3 and bank 1 off E1 of the same bit. SRC/DST codes 8-15 are
bank 1; word() derives the bank bit FROM the code, so a caller cannot select
SP_LO and forget to switch banks.

MISC IS NOW FULL. U29's O5/O7 were the last two free codes and the stack
spends both. O0 is the NONE slot and can never be reclaimed.

Deviations from dino_hardware_growth_plan.md, corrected inline there:

  - SRC3/DST3/MISC3 -> ~{SRC_BANK}/~{DST_BANK}/~{MISC_BANK}. A '138 has three
    address pins; the new bit is an ENABLE, not a fourth.
  - COND[2:0] -> FLAG_SEL0/FLAG_SEL1/FLAG_POL. COND0 loses KiCad's alias sort
    to CW21, steals the net off the CW bus, and produces net_not_bus_member.
  - CIN is a SELECT, not a carry value: one ROM bit cannot BE the carry.
  - MISC had two free codes, not three, and SP_LOAD is a DST d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
Other:
- added sheet Stack Pointer (stack_pointer.kicad_sch)
Changed lines of the file:
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@@
+	)
+	(sheet
+		(at 182.88 16.51)
+		(size 12.7 3.81)
+		(exclude_from_sim no)
+		(in_bom yes)
+		(on_board yes)
+		(dnp no)
+		(fields_autoplaced yes)
+		(stroke
+			(width 0.1524)
+			(type solid)
+		)
+		(fill
+			(color 0 0 0 0)
+		)
+		(property "Sheetname" "Stack Pointer"
+			(at 182.88 15.7984 0)
+			(show_name no)
+			(do_not_autoplace no)
+			(effects
+				(font
+					(size 1.27 1.27)
+				)
+				(justify left bottom)
+			)
+		)
+		(property "Sheetfile" "stack_pointer.kicad_sch"
+			(at 182.88 20.9046 0)
+			(show_name no)
+			(do_not_autoplace no)
+			(effects
+				(font
+					(size 1.27 1.27)
+				)
+				(justify left top)
+			)
+		)
+		(instances
+			(project "dino_v0_0_2"
+				(path "/e43166a5-d972-471d-b3cf-9f4f12c7f541"
+					(page "11")
+				)
+			)
+		)
 	)
 	(sheet

Commit message: feat: phase D on silicon — the machine executes from RAM
PROG_ramexec returns 0x6E. The PC has been above 0x7FFF and FETCH_RAM has
been high, both for the first time in this machine's life.

The missing condition was never "is this a fetch." ~ROM_OUT is asserted for
every src=ROM — opcode fetch, LDAI's immediate, LDA/STA/JMP/CALL operand
bytes — so an instruction living in RAM must read its operands from RAM
too. The condition is "a ROM-side read was requested, but the address is
above 0x7FFF":

    FETCH_RAM = NOR(~ROM_OUT, ~RAM_EN)

Six gate sections, no new IC. All six were free on U22/U37/U39, already in
sockets on the MDR board, where ~ROM_OUT and ~RAM_OUT already sit feeding
READS_IDLE. Only ~RAM_EN had to be brought in.

    U22 g3   FETCH_RAM     = NOR(~ROM_OUT, ~RAM_EN)
    U22 g4   ROM_BUF_ON    = NOR(~ROM_OUT, FETCH_RAM)
    U37 inv4 ~{FETCH_RAM}
    U37 inv6 ~{ROM_BUF_EN} = OR(~ROM_OUT, FETCH_RAM)   -> U19.19
    U37 inv5 ~{RAM_OE_G}   = AND(~RAM_OUT, ~FETCH_RAM) -> U26.22 + U51.9
    U39 g4   RAM_OE_ON     = NAND(~RAM_OUT, ~FETCH_RAM)

Two pin lifts on the memory board, eleven wires. U24.22 stays on ~ROM_OUT:
U24's own ~CE = M15 already deselects the ROM chip at RAM addresses.

Gating ~RAM_OUT upstream is what keeps this at six gates rather than eight.
U51 is a 7400 computing ~RAM_MDR_EN = AND(~RAM_OUT, ~WRITE_DIR), so one
gate on ~RAM_OUT moves both the RAM chip's ~OE and its buffer's ~CE.

Re-proved before building: all 15 src=ROM microcode rows carry mux_pc=True,
FETCH included, and FILL is src=NONE. A ROM-side read can now land in RAM,
so the standing "ROM reads are exempt from the src=RAM -> MAR loop" rule was
no longer free. It holds — MAR never drives M during a ROM-side read, and a
runaway opcode cannot open the loop either.

The witness is not permutation-blind. If the fetch had still come from ROM,
PC=0x9000 presents A0-A14 = 0x1000 to U24, which is 0xFF fill, which is
HALT, so the poison would have survived as 0xFF. 0x6E is 0x8B - 0x1D,
compu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
Other:
- note added: "MODULE CONTRACT — generated, do not hand-edit (kicad_contracts.py --stamp) IN: CW12=END, CW15=HALT <- Microcode_Decoder OUT: ~{RESET} -> ALU Module OUT: CLK -> ALU Module, Memory Address Regiser, Memory Data Register, Program Counter, Register Modules, Stack Pointer OUT: ~{CLK} -> ALU Module, Memory, Program Counter OUT: T0-3 -> Microcode_Decoder OUT: RESET -> Program Counter"
- note removed: "MODULE CONTRACT — generated, do not hand-edit (kicad_contracts.py --stamp) IN: CW12=END, CW15=HALT <- Microcode_Decoder OUT: ~{RESET} -> ALU Module OUT: CLK -> ALU Module, Memory Address Regiser, Memory Data Register, Program Counter, Register Modules OUT: ~{CLK} -> ALU Module, Memory, Program Counter OUT: T0-3 -> Microcode_Decoder OUT: RESET -> Program Counter"
Changed lines of the file:
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@@
 		(comment 4 "A Turing-Complete 8-bit \"Computer\"")
 	)
-	(text "MODULE CONTRACT — generated, do not hand-edit (kicad_contracts.py --stamp)\nIN: CW12=END, CW15=HALT <- Microcode_Decoder\nOUT: ~{RESET} -> ALU Module\nOUT: CLK -> ALU Module, Memory Address Regiser, Memory Data Register, Program Counter, Register Modules\nOUT: ~{CLK} -> ALU Module, Memory, Program Counter\nOUT: T0-3 -> Microcode_Decoder\nOUT: RESET -> Program Counter"
-		(exclude_from_sim no)
-		(at 156.718 170.942 0)
-		(effects
-			(font
-				(size 1.27 1.27)
-			)
-			(justify left bottom)
-		)
-	)
 	(junction
 		(at 133.35 74.93)
@@
 	)
 	(embedded_fonts no)
+	(text "MODULE CONTRACT — generated, do not hand-edit (kicad_contracts.py --stamp)\nIN: CW12=END, CW15=HALT <- Microcode_Decoder\nOUT: ~{RESET} -> ALU Module\nOUT: CLK -> ALU Module, Memory Address Regiser, Memory Data Register, Program Counter, Register Modules, Stack Pointer\nOUT: ~{CLK} -> ALU Module, Memory, Program Counter\nOUT: T0-3 -> Microcode_Decoder\nOUT: RESET -> Program Counter"
+		(exclude_from_sim no)
+		(at 156.718 170.942 0)
+		(effects
+			(font
+				(size 1.27 1.27)
+			)
+			(justify left bottom)
+		)
+	)
 )

Commit message: feat: phase E step A -- the 16K I/O window, in schematic
Carves 0x4000-0x7FFF out of ROM space and publishes a bus. The ROM now
answers 0x0000-0x3FFF only; the window decodes to no core chip, so W
reads its park -- 0xFF, which is HALT.

TWO NEW PACKAGES, both on the memory board:

  U74 '00  ~{M14}      = NAND(M14, M14)
           ~{ROM_SEL}  = NAND(~{RAM_EN}, ~{M14})
           ~{RAM_OE_G} = NAND(RAM_OE_ON, M15)
           ~{IO_SEL}   = NAND(~{RAM_EN}, M14)
  U75 '32  ~{IO_RD}    = OR(~{IO_SEL}, READS_IDLE)
           ~{IO_WR}    = OR(~{IO_SEL}, ~{RAM_WRITE_EN})
           RESET_B     = OR(RESET, GND)
           ~{IO_RD_Q}  = OR(~{IO_RD}, CLK)

Eight copper changes: U24.20 and U22.12 to ~{ROM_SEL}, U26.22/U51.9 fed
from U74 g3, U39.10 to ~{IO_RD}, U37.10 and U28.7 unlanded, U37.11 to
GND. Park: R4-R8 + R25-R27, 4.7k on W0-7. CLK crosses through R3, 100R,
source end -- the R2 treatment.

IN RETIRES. ~{SW_OUT} has zero pins project-wide. SWITCH-GATE1's enables
are strapped +5V until card zero drives them from an address decode.

THE ROM_EN ALIAS IS DELETED. Once U24.20 moved, ROM_EN named a net with
no ROM consumer. Deleting it half-way SPLIT the net and alias_splits()
caught it mid-edit -- M15: ['M15', 'M15/ROM_EN'], the exact two-key
failure that once cost this project the ROM chip-enable on every
continuity checklist ever generated.

CLK WAS A FOURTH CROSSING THE SPEC DID NOT CARRY. Census: 15 CLK pins,
none on the memory board; ~{CLK} at U51.4 is the wrong polarity and both
new packages are full. SECTION 1's cost table predated the read-term
split that spent U75 g4, so memory is +4 and MDR is +4 -- the wire margin
is zero. Ruled: stay on memory, the output-load argument still holds.

SWITCH-GATE1/SW1/R17-R24/C48 move to their own input.kicad_sch so the
DIP card is modelled as a card. No renumbering: 168 designators
unchanged, --since reports annotate=0.

TOOLING RECONCILED TO THE DESIGN, not the reverse:
  test_continuity_completeness  M15_PINS U24.20 -> U74.10; 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
Other:
- added sheet Input (input.kicad_sch)
- note added: "MODULE CONTRACT — generated, do not hand-edit (kicad_contracts.py --stamp) IN: CW12=END, CW15=HALT <- Microcode_Decoder OUT: ~{RESET} -> ALU Module OUT: CLK -> ALU Module, Memory, Memory Address Regiser, Memory Data Register, Program Counter, Register Modules, Stack Pointer OUT: ~{CLK} -> ALU Module, Memory, Program Counter OUT: RESET -> Memory, Program Counter OUT: T0-3 -> Microcode_Decoder"
- note removed: "MODULE CONTRACT — generated, do not hand-edit (kicad_contracts.py --stamp) IN: CW12=END, CW15=HALT <- Microcode_Decoder OUT: ~{RESET} -> ALU Module OUT: CLK -> ALU Module, Memory Address Regiser, Memory Data Register, Program Counter, Register Modules, Stack Pointer OUT: ~{CLK} -> ALU Module, Memory, Program Counter OUT: T0-3 -> Microcode_Decoder OUT: RESET -> Program Counter"
Changed lines of the file:
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@@
+		)
+	)
+	(sheet
+		(at 237.49 58.42)
+		(size 12.7 3.81)
+		(exclude_from_sim no)
+		(in_bom yes)
+		(on_board yes)
+		(dnp no)
+		(stroke
+			(width 0.1524)
+			(type solid)
+		)
+		(fill
+			(color 0 0 0 0)
+		)
+		(property "Sheetname" "Input"
+			(at 237.49 57.658 0)
+			(show_name no)
+			(do_not_autoplace no)
+			(effects
+				(font
+					(size 1.27 1.27)
+				)
+				(justify left bottom)
+			)
+		)
+		(property "Sheetfile" "input.kicad_sch"
+			(at 237.236 63.246 0)
+			(show_name no)
+			(do_not_autoplace no)
+			(effects
+				(font
+					(size 1.27 1.27)
+				)
+				(justify left top)
+			)
+		)
+		(instances
+			(project "dino_v0_0_2"
+				(path "/e43166a5-d972-471d-b3cf-9f4f12c7f541"
+					(page "12")
+				)
+			)
 		)
 	)
@@
 	)
 	(embedded_fonts no)
-	(text "MODULE CONTRACT — generated, do not hand-edit (kicad_contracts.py --stamp)\nIN: CW12=END, CW15=HALT <- Microcode_Decoder\nOUT: ~{RESET} -> ALU Module\nOUT: CLK -> ALU Module, Memory Address Regiser, Memory Data Register, Program Counter, Register Modules, Stack Pointer\nOUT: ~{CLK} -> ALU Module, Memory, Program Counter\nOUT: T0-3 -> Microcode_Decoder\nOUT: RESET -> Program Counter"
+	(text "MODULE CONTRACT — generated, do not hand-edit (kicad_contracts.py --stamp)\nIN: CW12=END, CW15=HALT <- Microcode_Decoder\nOUT: ~{RESET} -> ALU Module\nOUT: CLK -> ALU Module, Memory, Memory Address Regiser, Memory Data Register, Program Counter, Register Modules, Stack Pointer\nOUT: ~{CLK} -> ALU Module, Memory, Program Counter\nOUT: RESET -> Memory, Program Counter\nOUT: T0-3 -> Microcode_Decoder"
 		(exclude_from_sim no)
 		(at 156.718 170.942 0)
