File: dino_v0_0_2/alu.kicad_sch (KiCad schematic)
At the start: 0 parts

Commit message: v0.3.0 - Rev 1.2.0 Update
Other:
- note added: "We need to implement two TMP_A and TMP_B latches as "Shadow Latches""
- note added: "We need to introduce an extra ALU latch since Reg A can be an operand and resultant. We plan to have A store the result, so there's a step in between"
- title: Dino v0.0.2 -> Dino v0.0.3
Changed lines of the file:
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@@
 (kicad_sch
-	(version 20250114)
+	(version 20260306)
 	(generator "eeschema")
-	(generator_version "9.0")
+	(generator_version "10.0")
 	(paper "USLetter")
 	(title_block
-		(title "Dino v0.0.2")
-		(date "2025-08-14")
-		(rev "v1.1.0")
+		(title "Dino v0.0.3")
+		(date "2026-07-12")
+		(rev "v1.2.0")
 		(comment 3 "An 8-bit computer with 16-bit addressing and 16-bit control words")
 		(comment 4 "A Turing-Complete 8-bit \"Computer\"")
 	)
+	(text "We need to implement two TMP_A and TMP_B latches as \"Shadow Latches\""
+		(exclude_from_sim no)
+		(at 86.36 93.726 0)
+		(effects
+			(font
+				(size 1.27 1.27)
+			)
+		)
+	)
+	(text "We need to introduce an extra ALU latch \nsince Reg A can be an operand and resultant. \nWe plan to have A store the result, so there's a step in between\n"
+		(exclude_from_sim no)
+		(at 85.598 83.058 0)
+		(effects
+			(font
+				(size 1.27 1.27)
+			)
+		)
+	)
 )
