File: dino_v0_0_2/mdr.kicad_sch (KiCad schematic)
At the start: 15 parts, among them SW2 SW_Push, SW3 SW_Push, U18 74LS373, U22 74LS121, U23 74LS244N, U25 74LS245, U34 74LS373, U37 74LS04, U38 74LS74, U39 74LS00, U52 74LS32

Commit message: v0.3.0 - Rev 1.2.0 Update
Parts:
- removed C17: 100pF, symbol Device:C_Small
- removed R3, R5: R, symbol Device:R
- removed R6: 2.2kΩ, symbol Device:R
- removed SW2, SW3: SW_Push, symbol Switch:SW_Push
- removed U22: 74LS121, symbol 74xx:74LS121
- removed U23: 74LS244N, symbol 74xx:74LS244N
- removed U38: 74LS74, symbol 74xx:74LS74
- removed U52: 74LS32, symbol 74xx:74LS32
- added U22: 74LS02, symbol 74xx:74LS02
Connections:
- net +5V: now also U22.14 (VCC)
- net CLK: now also U22.2
- net GND: now also U22.7 (GND)
- net MDR_OUT: now also U37.6, U22.6; no longer U37.3
- net ~{IR_LOAD}: now also U22.3; no longer U34.11 (LE), U39.6
- net ~{MDR_OUT}: now also U37.5; no longer U25.1 (DIR), U37.4
- net ~{RAM_LOAD}: now reaches U39.4
- net ~{RAM_LOAD}: now also U37.3; no longer U39.2
- net at U37.1: now also U39.3
- net READS_IDLE: now reaches U37.2
- net READS_IDLE: now also U39.5
- net IR_LE: no longer names the net of U39.9
- net IR_LE: no longer U39.5
- net IR_PULSE: no longer names the net of U39.8
- net MDR_LOAD: no longer names the net of U39.13
- net MDR_LOAD: no longer U39.1
- net MDR_PULSE: no longer names the net of U39.11
- net PULSE_REQ: no longer names the net of U39.12
- net PULSE_REQ: no longer U39.10
- net RESET renamed ~{MDR_EN}
- net ~{MDR_EN}: now also U22.4
- net ~{MDR_LOAD} renamed LE_MDR
- net LE_MDR: now also U39.6, U22.5; no longer U39.3
- new net LE_IR: U22.1, U34.11 (LE)
- new net WRITE_DIR: U25.1 (DIR), U37.4
- new net ~{RAM_OUT}: U39.2
- new net ~{ROM_OUT}: U39.1
- no-connect marks 27 -> 18
Other:
- title: Dino v0.0.2 -> Dino v0.0.3
- moved on the sheet: U18, U25, U34, U37A, U37B, U37C, U37D, U37E, U37F, U37G, U39C, U39D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
