File: dino_v0_0_2/mdr.kicad_sch (KiCad schematic)
At the start: 6 parts, among them U18 74LS373, U22 74LS02, U25 74LS245, U34 74LS373, U37 74LS04, U39 74LS00

Commit message: DINO v0.0.3: complete ALU/control-word, add MAR+reset sheets, wire reset circuit
ALU sheet: flags register moved from '173 (not in stock) to '273 + a '157
mux to emulate the missing load-enable pins; Z-detect built from a NOR+AND
De Morgan tree instead of a '260; ALU_CIN built from NAND(SA1,SA0) reusing
two already-placed spare gates instead of a dedicated XOR/'86. Sheet is
now fully wired and netlist-clean.

Control word sheet: all 16 CW bits assigned and wired (3x '138 decoders
for the load/source/misc fields, direct bus taps for HALT/PC_MAR_MUX/
PC_UP/END and the ALU SA[2:0] select). Found and fixed several cross-
sheet signal-name mismatches this uncovered (OUT_REG_LOAD/REG_OUT_LOAD,
PC_MAR_MUX/PC_MUX, T-state counter labels, a mirror-reversed IRB->ROM-
address buffer in microcode).

New: MAR and reset sheets, wired into the root hierarchy. Reset circuit
is a from-scratch design: RC+button+74HC14 Schmitt front end feeds the
async PRESET of the clock cluster's spare '74 half (U27B), synchronizing
release to CLK; its Q/~Q fan out to the flags register, the T-state
counter's clear, and (OR'd with the existing microcode-driven PC_CLEAR,
reusing spare gates on the same '02) the PC counters' clear.

Deprecated 7 schematic files no longer referenced by the root sheet's
hierarchy into dino_v0_0_2/deprecated/. Added docs/notes/kicad_netlist.py,
a .kicad_sch connectivity auditor (pin/net resolution incl. buses and
same-name local-label merging) used throughout this session to find the
above bugs; archived completed-work docs into docs/notes/Done/ and
rewrote dino_session_state.md as the current authoritative state+TODO.

Co-Authored-By: Claude Sonnet 5 <noreply@anthropic.com>
Parts:
- added C27, C28, C29, C30, C31, C32: 0.1µF, symbol Device:C_Small
Connections:
- net +5V: now also C27.1, C28.1, C29.2, C30.1, C31.1, C32.2
- net GND: now also C27.2, C28.2, C29.1, C30.2, C31.2, C32.1
- net MDR7: now reaches U25.11 (B7)
- net MDR7: now also U18.18 (D7), U18.19 (O7)
- net MDR6: now reaches U25.12 (B6)
- net MDR6: now also U18.16 (O6), U18.17 (D6)
- net MDR5: now reaches U25.13 (B5)
- net MDR5: now also U18.14 (D5), U18.15 (O5)
- net MDR4: now reaches U25.14 (B4)
- net MDR4: now also U18.12 (O4), U18.13 (D4)
- net MDR3: now reaches U25.15 (B3)
- net MDR3: now also U18.8 (D3), U18.9 (O3)
- net MDR2: now reaches U25.16 (B2)
- net MDR2: now also U18.6 (O2), U18.7 (D2)
- net MDR1: now reaches U25.17 (B1)
- net MDR1: now also U18.4 (D1), U18.5 (O1)
- net MDR0: now reaches U25.18 (B0)
- net MDR0: now also U18.2 (O0), U18.3 (D0)
- net W0: now reaches U25.2 (A0)
- net W0: now also U34.3 (D0)
- net W1: now reaches U25.3 (A1)
- net W1: now also U34.4 (D1)
- net W2: now reaches U25.4 (A2)
- net W2: now also U34.7 (D2)
- net W3: now reaches U25.5 (A3)
- net W3: now also U34.8 (D3)
- net W4: now reaches U25.6 (A4)
- net W4: now also U34.13 (D4)
- net W5: now reaches U25.7 (A5)
- net W5: now also U34.14 (D5)
- net W6: now reaches U25.8 (A6)
- net W6: now also U34.17 (D6)
- net W7: now reaches U25.9 (A7)
- net W7: now also U34.18 (D7)
- net IRB4: now reaches U34.12 (O4)
- net IRB5: now reaches U34.15 (O5)
- net IRB6: now reaches U34.16 (O6)
- net IRB7: now reaches U34.19 (O7)
- net IRB0: now reaches U34.2 (O0)
- net IRB1: now reaches U34.5 (O1)
- net IRB2: now reaches U34.6 (O2)
- net IRB3: now reaches U34.9 (O3)
Other:
- note removed: "Data Bus"
- note removed: "MDR Bus"
