File: dino_v0_0_2/program_counter.kicad_sch (KiCad schematic)
At the start: 18 parts, among them U1 74LS193, U10 74LS04, U11 74LS245, U12 74LS245, U13 74LS245, U14 74LS245, U2 74LS193, U3 74LS193, U4 74LS193

Commit message: v0.3.0 - Rev 1.2.0 Update
Other:
- title: Dino v0.0.2 -> Dino v0.0.3
