File: dino_v0_0_2/reg_logic.kicad_sch (KiCad schematic)
At the start: 11 parts, among them U57 74LS02, U58 74LS121, U62 74LS00, U63 74LS00, U64 74LS121, U65 74LS04, U66 74LS02

Commit message: v0.3.0 - Rev 1.2.0 Update
Parts:
- removed C20, C21: 100pF, symbol Device:C_Small
- removed R25, R26: 2.2kΩ, symbol Device:R
- removed U57, U66: 74LS02, symbol 74xx:74LS02
- removed U58, U64: 74LS121, symbol 74xx:74LS121
- removed U62, U63: 74LS00, symbol 74xx:74LS00
- removed U65: 74LS04, symbol 74xx:74LS04
Connections:
- no-connect marks 8 -> 0
Other:
- title: Dino v0.0.2 -> Dino v0.0.3
