File: dino_v0_0_2/registers_a_b.kicad_sch (KiCad schematic)
At the start: 22 parts, among them U31 74LS373, U32 74LS373, U33 74LS373, U35 74LS373, U41 74LS245, U42 74LS245, U43 74LS245, U44 74LS245, U5 74LS08, U57 74LS02, U66 74LS02

Commit message: Machine Complete
All ten DINO modules bench-proven on the ATmega2560 rig: root, pc,
microcode, control_word, mdr, registers, mar, memory, alu, io. Coverage
lint reports 0 gaps and 0 pending.

Test modules (mod_*.c) plus host-tested expect models (cw/mdr/reg/mar/
mem/alu_expect.h) — pure logic, no AVR headers, exhaustive host tests
written RED before any bench run. Every assertion was netlist-verified
against the schematic before it was encoded.

Generators, so no table is hand-maintained:
  kicad_contracts.py   contracts + pinmap from the KiCad netlist
  microcode_gen.py     microcode ROM images
  progrom_gen.py       program ROM (DIAG + the milestone program)
  layout_gen.py        breadboard placement, slot maps, wiring guides

Two house rules learned the hard way and now codified in BRINGUP.md:
  mirror-witness   a write-then-read through one bus bank is
                   permutation-blind; every module needs an asymmetric
                   path (this is what caught the flipped PORTF->MDR bank)
  phantom power    rig lines feed DUT VCC through input clamp diodes, so
                   an unpowered board reads fine; every module gets a
                   power test holding outputs at the non-sourcing level

The ALU slot map in layout_gen.py is AS-BUILT and FROZEN — read off the
strip by beeping each slot to its chip pin, not derived. Once a strip is
populated its slot map is copper.

Housekeeping: .gitignore for __pycache__, KiCad .lck, Obsidian workspace
state, and compiled host-test binaries; those are untracked here.

Next: the integration ladder (INT-A/B/B2/C/D/E), then free-run of
LDAI 5; LDBI 3; ADD; OUT; HALT — the milestone, where the machine adds
two numbers.

Co-Authored-By: Claude Opus 5 (1M context) <noreply@anthropic.com>
Parts:
- removed unit 5 of U66
- renumbered U66 to U57

Commit message: feat: phase D on silicon — the machine executes from RAM
PROG_ramexec returns 0x6E. The PC has been above 0x7FFF and FETCH_RAM has
been high, both for the first time in this machine's life.

The missing condition was never "is this a fetch." ~ROM_OUT is asserted for
every src=ROM — opcode fetch, LDAI's immediate, LDA/STA/JMP/CALL operand
bytes — so an instruction living in RAM must read its operands from RAM
too. The condition is "a ROM-side read was requested, but the address is
above 0x7FFF":

    FETCH_RAM = NOR(~ROM_OUT, ~RAM_EN)

Six gate sections, no new IC. All six were free on U22/U37/U39, already in
sockets on the MDR board, where ~ROM_OUT and ~RAM_OUT already sit feeding
READS_IDLE. Only ~RAM_EN had to be brought in.

    U22 g3   FETCH_RAM     = NOR(~ROM_OUT, ~RAM_EN)
    U22 g4   ROM_BUF_ON    = NOR(~ROM_OUT, FETCH_RAM)
    U37 inv4 ~{FETCH_RAM}
    U37 inv6 ~{ROM_BUF_EN} = OR(~ROM_OUT, FETCH_RAM)   -> U19.19
    U37 inv5 ~{RAM_OE_G}   = AND(~RAM_OUT, ~FETCH_RAM) -> U26.22 + U51.9
    U39 g4   RAM_OE_ON     = NAND(~RAM_OUT, ~FETCH_RAM)

Two pin lifts on the memory board, eleven wires. U24.22 stays on ~ROM_OUT:
U24's own ~CE = M15 already deselects the ROM chip at RAM addresses.

Gating ~RAM_OUT upstream is what keeps this at six gates rather than eight.
U51 is a 7400 computing ~RAM_MDR_EN = AND(~RAM_OUT, ~WRITE_DIR), so one
gate on ~RAM_OUT moves both the RAM chip's ~OE and its buffer's ~CE.

Re-proved before building: all 15 src=ROM microcode rows carry mux_pc=True,
FETCH included, and FILL is src=NONE. A ROM-side read can now land in RAM,
so the standing "ROM reads are exempt from the src=RAM -> MAR loop" rule was
no longer free. It holds — MAR never drives M during a ROM-side read, and a
runaway opcode cannot open the loop either.

The witness is not permutation-blind. If the fetch had still come from ROM,
PC=0x9000 presents A0-A14 = 0x1000 to U24, which is 0xFF fill, which is
HALT, so the poison would have survived as 0xFF. 0x6E is 0x8B - 0x1D,
compu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
Other:
- note added: "MODULE CONTRACT — generated, do not hand-edit (kicad_contracts.py --stamp) IN: ~{REG_A_LOAD}, ~{REG_A_OUT}, ~{REG_B_LOAD}, ~{REG_B_OUT}, ~{REG_C_LOAD}, ~{REG_C_OUT}, ~{REG_OUT_LOAD} <- Control Word Module IN: CLK <- root OUT: MDR0-7 -> Memory, Memory Data Register, Stack Pointer OUT: OB0-7 -> Output"
- note removed: "MODULE CONTRACT — generated, do not hand-edit (kicad_contracts.py --stamp) IN: ~{REG_A_LOAD}, ~{REG_A_OUT}, ~{REG_B_LOAD}, ~{REG_B_OUT}, ~{REG_C_LOAD}, ~{REG_C_OUT}, ~{REG_OUT_LOAD} <- Control Word Module IN: CLK <- root OUT: MDR0-7 -> Memory, Memory Data Register OUT: OB0-7 -> Output"
Changed lines of the file:
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@@
 		)
 	)
-	(text "MODULE CONTRACT — generated, do not hand-edit (kicad_contracts.py --stamp)\nIN: ~{REG_A_LOAD}, ~{REG_A_OUT}, ~{REG_B_LOAD}, ~{REG_B_OUT}, ~{REG_C_LOAD}, ~{REG_C_OUT}, ~{REG_OUT_LOAD} <- Control Word Module\nIN: CLK <- root\nOUT: MDR0-7 -> Memory, Memory Data Register\nOUT: OB0-7 -> Output"
-		(exclude_from_sim no)
-		(at 146.558 169.926 0)
-		(effects
-			(font
-				(size 1.27 1.27)
-			)
-			(justify left bottom)
-		)
-	)
 	(junction
 		(at 196.85 142.24)
@@
 		)
 	)
+	(text "MODULE CONTRACT — generated, do not hand-edit (kicad_contracts.py --stamp)\nIN: ~{REG_A_LOAD}, ~{REG_A_OUT}, ~{REG_B_LOAD}, ~{REG_B_OUT}, ~{REG_C_LOAD}, ~{REG_C_OUT}, ~{REG_OUT_LOAD} <- Control Word Module\nIN: CLK <- root\nOUT: MDR0-7 -> Memory, Memory Data Register, Stack Pointer\nOUT: OB0-7 -> Output"
+		(exclude_from_sim no)
+		(at 146.558 169.926 0)
+		(effects
+			(font
+				(size 1.27 1.27)
+			)
+			(justify left bottom)
+		)
+	)
