File: dino_v0_0_2/dino_v0_0_2.kicad_pcb (KiCad board)
At the start: 2 copper layers, 389.3 x 410.1 mm, 198 parts, among them J10 PS_ON, J9 ATX-24, SW1 SW_DIP_x08, SW2 RESET_BTN, U1 74LS193, U10 74LS02, U11 74LS245, U12 74LS245, U13 74LS245, U14 74LS245, U15 AT28C64B, U16 74LS244N, U17 74LS244N, U18 74LS373, U19 74LS245, U2 74LS193, U20 74LS163, U21 74LS245, U22 74LS02, U23 AT28C64B, U24 AT28C256, U25 74LS245, U26 MCM60256AP, U27 74LS74, U28 74LS138, U29 74LS138, U3 74LS193, U30 74LS138, U31 74LS373, U32 74LS373, U33 74LS373, U34 74LS373, U35 74LS373, U36 7400, U37 74LS04, U38 74F382N, U39 74LS00, U4 74LS193, U40 74F382N, U41 74LS245, U42 74LS245, U43 74LS245, U44 74LS245, U45 74LS373, U46 74LS373, U47 74LS373, U48 74LS157, U49 74LS273, U5 74LS08, U50 74LS02, U51 7400, U52 74LS02, U53 74LS08, U54 74LS245, U55 74LS373, U56 74LS14, U57 74LS02, U58 74LS373, U59 74LS245, U6 74LS163, U60 74LS02, U61 74LS02, U62 74LS02, U63 74LS169, U64 74LS169, U65 74LS169, U66 74LS169, U67 74LS245, U68 74LS245, U69 74LS08, U7 74LS138, U70 74LS138, U71 74LS138, U72 74LS245, U73 74LS245, U74 74LS00, U75 74LS32, U76 74LS138, U77 74LS157, U8 74LS138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

Commit message: feat(kicad): peripheral bus sheet, dino_io card project, dino_bus lib
Eight 2x25 0.1in card-edge sockets on the core (peripheral_bus.kicad_sch,
J1-J8) bussed on global labels; U78 '04 buffers ~{CLK} into CLK_B so no
card sees U27.5 raw; ~{IRQ} ~{NMI} ~{DMARQ} ~{DMAAK} RDY named and
reserved, spares no-connected. Rails are what the picoPSU delivers.

Card zero leaves the core: the Input sheet becomes dino_io/, references
unchanged, plus edge connector J1. input_output.kicad_sch is now
front_panel.kicad_sch: the OB LEDs are the OUT register's display, not a
card, and the W park stays at the origin (PHASE_E).

dino_bus/ is generated from one pin table in bus_gen.py: both symbol
flavours, the finger footprint, and a placeholder socket footprint until
a part is chosen. Edge-side pins carry direction types so a card project
passes ERC alone; socket side is passive.

Proof: core and card netlists joined through the slot-0 pin numbers
partition every pre-existing pin exactly as the core did before the
split. ERC 0/0 on both projects. dino_serial not yet given its J2.

Co-Authored-By: Claude Fable 5.1 <noreply@anthropic.com>
Claude-Session: https://claude.ai/code/session_018irreFHb1xEykW5kCD26ow
Parts:
- removed C48, C81: 0.1µF, Capacitor_THT:C_Disc_D5.0mm_W2.5mm_P2.50mm
- removed R17, R18, R19, R20, R21, R22, R23, R24: 10kΩ, Resistor_THT:R_Axial_DIN0207_L6.3mm_D2.5mm_P10.16mm_Horizontal
- removed SW1: SW_DIP_x08, Button_Switch_THT:SW_DIP_SPSTx08_Slide_9.78x22.5mm_W7.62mm_P2.54mm
- removed SWITCH-GATE1: 74LS244N, Package_DIP:DIP-20_W7.62mm
- removed U76: 74LS138, Package_DIP:DIP-16_W7.62mm
- added J1: DINO_BUS_SOCKET, dino_bus:EdgeSocket_2x25_P2.54mm_THT, F.Cu at (295.9, 33.3)
- added J2: DINO_BUS_SOCKET, dino_bus:EdgeSocket_2x25_P2.54mm_THT, F.Cu at (295.9, 51.1)
- added J3: DINO_BUS_SOCKET, dino_bus:EdgeSocket_2x25_P2.54mm_THT, F.Cu at (295.9, 68.8)
- added J4: DINO_BUS_SOCKET, dino_bus:EdgeSocket_2x25_P2.54mm_THT, F.Cu at (295.9, 86.6)
- added J5: DINO_BUS_SOCKET, dino_bus:EdgeSocket_2x25_P2.54mm_THT, F.Cu at (295.9, 104.4)
- added J6: DINO_BUS_SOCKET, dino_bus:EdgeSocket_2x25_P2.54mm_THT, F.Cu at (295.9, 122.2)
- added J7: DINO_BUS_SOCKET, dino_bus:EdgeSocket_2x25_P2.54mm_THT, F.Cu at (295.9, 140.0)
- added J8: DINO_BUS_SOCKET, dino_bus:EdgeSocket_2x25_P2.54mm_THT, F.Cu at (295.9, 157.7)
- added U78: 74LS04, Package_DIP:DIP-14_W7.62mm, F.Cu at (262.9, 5.08)
- moved C60 331.7 mm to (17.8, 405.0)
- moved C61 331.7 mm to (30.5, 405.0)
- moved C62 331.7 mm to (43.2, 405.0)
- moved C63 331.7 mm to (55.9, 405.0)
- moved U54 331.7 mm to (2.54, 371.7)
- moved U55 331.7 mm to (17.8, 371.7)
- moved U58 331.7 mm to (33.0, 371.7)
- moved U59 331.7 mm to (48.3, 371.7)
- moved U60 331.7 mm to (63.5, 371.7)
- moved C59 331.7 mm to (5.08, 405.0)
- moved C11 315.2 mm to (55.9, 249.1)
- moved C12 315.2 mm to (68.6, 249.1)
- moved C13 315.2 mm to (81.3, 249.1)
- moved C14 315.2 mm to (94.0, 249.1)
- moved C15 315.2 mm to (106.7, 249.1)
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Connections:
- net /Memory/~{IO_SEL} renamed ~{IO_SEL}
- U75 pad 6: /Memory/~{IO_WR} -> ~{IO_WR}
- U75 pad 8: /Memory/RESET_B -> RESET_B
Other:
- board size 389.3 x 410.1 mm -> 374 x 523.9 mm

Commit message: feat(pcb): place and route the mainboard, 299x223 2-layer
Draft was 374x524 with nothing routed. Placement by simulated annealing
over a DIP cell grid (HPWL, clock weighted), then hand-trimmed: LEDs and
their 330R leave the board for an OB header J11, W park resistors sit at
the slot-column end, slots J1-J8 respaced to 20.32 mm. Freerouting 2.4.1
on KiCad's own DSN export with the netclasses (Default 0.25, PWR 1.0,
CLK 0.3); GND pours both layers plus router-placed GND bridges. kicad-cli
DRC: 0 unconnected, 0 clearance, 0 shorts; 38 starved-thermal (per-layer
check) and silk warnings remain.

docs/notes/test_pcb_envelope.py enforces the card-edge mechanics against
the saved board: 8 slots in one column at 20.32 mm, no part taller than a
DIP under a card overhang, and CLK/~CLK/CLK_B copper within +20% of the
routed baseline.

Co-Authored-By: Claude Opus 5 <noreply@anthropic.com>
Claude-Session: https://claude.ai/code/session_01Qfuso4zXCFF2iuVHgVo7c8
Parts:
- removed D1, D2, D3, D4, D5, D6, D7, D8: LED, LED_THT:LED_D5.0mm
- removed R10, R11, R12, R13, R14, R15, R16, R9: 330Ω, Resistor_THT:R_Axial_DIN0207_L6.3mm_D2.5mm_P10.16mm_Horizontal
- added J11: Conn_01x08_Socket, Connector_PinSocket_2.54mm:PinSocket_1x08_P2.54mm_Vertical, F.Cu at (3.08, 195.8)
- moved C42 503.5 mm to (150.7, 7.45)
- moved C43 462.2 mm to (178.9, 53.2)
- moved C64 460.7 mm to (57.0, 53.2)
- moved C41 445.4 mm to (209.4, 88.7)
- moved C38 433.9 mm to (209.4, 119.2)
- moved C28 417.8 mm to (19.4, 7.45)
- moved C32 409.0 mm to (102.6, 7.45)
- moved U16 408.9 mm to (115.1, 11.4)
- moved C22 407.9 mm to (102.7, 53.2)
- moved U9 406.7 mm to (74.1, 11.4)
- moved C27 401.3 mm to (80.5, 7.45)
- moved C45 391.6 mm to (11.3, 119.2)
- moved R25 391.6 mm to (259.8, 15.1), turned to -90 degrees
- moved C46 391.1 mm to (26.5, 119.2)
- moved U23 387.6 mm to (196.0, 11.4)
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Routing:
- net GND: track 0.00 -> 3616.9 mm, vias 0 -> 4
- net +5V: track 0.00 -> 2331.1 mm, vias 0 -> 1
- net W1: track 0.00 -> 706.7 mm, vias 0 -> 3
- net W0: track 0.00 -> 688.7 mm, vias 0 -> 7
- net W2: track 0.00 -> 681.0 mm, vias 0 -> 6
- net W7: track 0.00 -> 670.0 mm, vias 0 -> 3
- net M14: track 0.00 -> 657.5 mm
- net M5: track 0.00 -> 650.3 mm, vias 0 -> 4
- net W5: track 0.00 -> 647.8 mm, vias 0 -> 4
- net M4: track 0.00 -> 645.2 mm, vias 0 -> 2
- net W6: track 0.00 -> 642.4 mm, vias 0 -> 3
- net M6: track 0.00 -> 623.0 mm, vias 0 -> 3
- net M2: track 0.00 -> 618.0 mm, vias 0 -> 8
- net M13: track 0.00 -> 617.9 mm, vias 0 -> 2
- net M12: track 0.00 -> 614.8 mm, vias 0 -> 3
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- added copper zone on B.Cu, net GND
- added copper zone on F.Cu, net GND
Other:
- board size 374 x 523.9 mm -> 298.9 x 222.8 mm
- board text added: "CARD OVERHANG STRIP x219-237 : NO PARTS : BUS CORRIDOR (test_pcb_envelope.py)"
- board text added: "SLOTS J1-J8 : 17.78mm PITCH : CARD 103.5 WIDE, HANGS 17.5 PAST EDGE : NO PART >8mm WITHIN 9mm OF A SLOT LINE"

Commit message: feat(pcb): started PCB — mainboard DRC clean, placer tools, serial card footprints
Mainboard (dino_v0_0_2): GND zones on both layers re-parameterised to
0.25 mm clearance / 0.2 mm min width so the pour threads the channels
the router spaced for 0.25 mm tracks; 43 GND jump vias and one F.Cu
rule area (J6 pad 50) clear the starved-thermal reports. kicad-cli DRC:
0 unconnected, 0 clearance, 0 shorts; silk warnings only. Project zone
defaults and via size follow.

docs/notes/pcb_tools: the placement scripts from the 2026-09-12 layout
session (anneal.py simulated-annealing cell placer, hpwl.py, report.py,
place_sheetrows.py), promoted verbatim from a session scratchpad so the
DMA/INT re-shuffle can reuse them. Throwaway quality; README says how.

dino_serial: footprints assigned to all six parts, card PCB started.

Co-Authored-By: Claude Opus 5 <noreply@anthropic.com>
Claude-Session: https://claude.ai/code/session_01Qfuso4zXCFF2iuVHgVo7c8
Routing:
- net GND: track 3616.9 -> 3669.0 mm, vias 4 -> 46
