File: dino_v0_0_2/dino_v0_0_2.kicad_pcb (KiCad board)
At the start: 4 copper layers, 298.9 x 270 mm, 202 parts, among them J1 DINO_BUS_SOCKET, J10 PS_ON, J11 Conn_01x08_Socket, J2 DINO_BUS_SOCKET, J3 DINO_BUS_SOCKET, J4 DINO_BUS_SOCKET, J5 DINO_BUS_SOCKET, J6 DINO_BUS_SOCKET, J7 DINO_BUS_SOCKET, J8 DINO_BUS_SOCKET, J9 ATX-24, SW2 RESET_BTN, U1 74LS193, U10 74LS02, U11 74LS245, U12 74LS245, U13 74LS245, U14 74LS245, U15 AT28C64B, U16 74LS244N, U17 74LS244N, U18 74LS373, U19 74LS245, U2 74LS193, U20 74LS163, U21 74LS245, U22 74LS02, U23 AT28C64B, U24 AT28C256, U25 74LS245, U26 MCM60256AP, U27 74LS74, U28 74LS138, U29 74LS138, U3 74LS193, U30 74LS138, U31 74LS373, U32 74LS373, U33 74LS373, U34 74LS373, U35 74LS373, U36 7400, U37 74LS04, U38 74F382N, U39 74LS00, U4 74LS193, U40 74F382N, U41 74LS245, U42 74LS245, U43 74LS245, U44 74LS245, U45 74LS373, U46 74LS373, U47 74LS373, U48 74LS157, U49 74LS273, U5 74LS08, U50 74LS02, U51 7400, U52 74LS02, U53 74LS08, U54 74LS245, U55 74LS373, U56 74LS14, U57 74LS02, U58 74LS373, U59 74LS245, U6 74LS163, U60 74LS02, U61 74LS02, U62 74LS02, U63 74LS169, U64 74LS169, U65 74LS169, U66 74LS169, U67 74LS245, U68 74LS245, U69 74LS08, U7 74LS138, U70 74LS138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

Commit message: feat(pcb): five grounded M3 mounting holes
H1-H5 (MountingHole_3.2mm_M3_Pad_Via, pad + stitching vias to the GND
plane) on the power sheet, pin 1 on GND. H1-H4 at the corners, 5 mm in
(H3 shifted to x 8.81 to clear J11); H5 at (85.88, 217.96), an interior
spot no track or part crosses, so the routing from 32aaa36 is unchanged.
KiCad DRC: 0 unconnected, 0 errors, 0 warnings, schematic parity 0.
ERC unchanged from the 2026-10-06 baseline.

Co-Authored-By: Claude Opus 5.5 <noreply@anthropic.com>
Claude-Session: https://claude.ai/code/session_01JGxSS4MVUcaZdKZGtKroSg
Parts:
- added H1: M3 GND, MountingHole:MountingHole_3.2mm_M3_Pad_Via, F.Cu at (5.00, 5.00)
- added H2: M3 GND, MountingHole:MountingHole_3.2mm_M3_Pad_Via, F.Cu at (293.9, 5.00)
- added H3: M3 GND, MountingHole:MountingHole_3.2mm_M3_Pad_Via, F.Cu at (8.81, 265.0)
- added H4: M3 GND, MountingHole:MountingHole_3.2mm_M3_Pad_Via, F.Cu at (293.9, 265.0)
- added H5: M3 GND, MountingHole:MountingHole_3.2mm_M3_Pad_Via, F.Cu at (85.9, 218.0)
