File: dino_io/dino_io.kicad_sch (KiCad schematic)
At the start: 14 parts, among them J1 DINO_BUS_EDGE, SW1 SW_DIP_x08, U76 74LS138

Commit message: feat(twin): netsim replaces the FPGA twin; host suite green
The Rev 1.0 netlist, the one the PCB is routed from, is now DINO's only
twin: netsim_gen.py emits one Verilog instance per chip, wired by pin
number, with no option to rewire. Icarus runs the burned ROMs on it.
make twin: 43 images x 3 power-up seeds, 129/129 match the oracle, HALT,
no unknown machine state, no RAM write under tWP. isa 0xB4, isasoak
0x00, carry 0xAD. test_netsim pins the Verilog to the netlist (1530
chip pins). The FPGA twin (fpga/, fpga_gen and its tests) is deleted.

Host suite: 656 passed, 0 failed, nothing ignored. The tests follow the
schematic as built:
- contracts: probe header J15, test points and DNP pads consume nothing
- continuity: a label shared between sheets is one net, as in KiCad
- footprint_gen knows the Rev 1.0 parts as placed on the audited board
- erc_cleanup merges exclusions and keys every alias-marker placement;
  mainboard ERC 0 violations (exclusion keys only, netlist unchanged)
- bus_gen.flatten tags card refs (card zero's U76 vs the ALU's U76)
- card zero's edge follows the 10-29 bus pinout: pin 1 CLK_B (NC),
  pin 17 GND; edge symbol re-embedded. Card project only, not in fab.
- serial card test: U104 7406N carries INTR onto ~{IRQ}
- block ladder and rig pinmap retired with their tests

Co-Authored-By: Claude Opus 5.5 <noreply@anthropic.com>
Connections:
- net GND: now also J1.17 (GND); no longer J1.1 (GND)
